File: hw/icenes.sch (KiCad schematic (older format))
At the start: 4 parts

Commit message: Added voltage generators for 3.3V, 1.2V and 5V. Added more info and footprints to some components. Connected signals to the NES connector to banks 0 and 1.
Parts:
- added C? (x3): C10uF, Capacitor_SMD:C_0603_1608Metric_Pad1.05x0.95mm_HandSolder, symbol icenes-library:C10uF
- added C? (x3): C22uF, Capacitor_SMD:C_0603_1608Metric_Pad1.05x0.95mm_HandSolder, symbol icenes-library:C22uF
- added C? (x2): C6.8pF, Capacitor_SMD:C_0603_1608Metric_Pad1.05x0.95mm_HandSolder, symbol icenes-library:C6.8pF
- added L? (x3): L10uH, Inductor_SMD:L_1206_3216Metric_Pad1.42x1.75mm_HandSolder, symbol icenes-library:L10uH
- added R?: R820K, Resistor_SMD:R_0603_1608Metric_Pad1.05x0.95mm_HandSolder, symbol icenes-library:R820K
- added R?: R91K, Resistor_SMD:R_0603_1608Metric_Pad1.05x0.95mm_HandSolder, symbol icenes-library:R91K
- added R? (x3): R1M, Resistor_SMD:R_0603_1608Metric_Pad1.05x0.95mm_HandSolder, symbol icenes-library:R1M
- added R?: R510K, Resistor_SMD:R_0603_1608Metric_Pad1.05x0.95mm_HandSolder, symbol icenes-library:R510K
- added R?: R360K, Resistor_SMD:R_0603_1608Metric_Pad1.05x0.95mm_HandSolder, symbol icenes-library:R360K
- added R? (x3): R0, Resistor_SMD:R_0805_2012Metric_Pad1.15x1.40mm_HandSolder, symbol icenes-library:R0
- added TP? (x9): TestPoint, symbol Connector:TestPoint
- added U? (x2): TPS62050, symbol icenes-library:TPS62050
- added U?: TPS62056, symbol icenes-library:TPS62056
- D?: footprint (none) -> Diode_SMD:D_0603_1608Metric_Pad1.05x0.95mm_HandSolder; Manufacturer (none) -> Comchip; Part number (none) -> CDBU0520
Connections:
- net labels added: +5V, USB_DM, USB_DP, Vin
- wire segments 55 -> 185
Other:
- moved on the sheet: D?, U?A

Commit message: GPIO headers for banks 2 and 3.
Parts:
- added C? (x15): C1uF, Capacitor_SMD:C_0603_1608Metric_Pad1.05x0.95mm_HandSolder, symbol icenes-library:C1uF
Connections:
- wire segments 185 -> 245

Commit message: Footprints.
Parts:
- U?: Manufacturer (none) -> Lattice; Part number (none) -> iCE40HX8K-CT256
- U? (x2): footprint (none) -> Package_SO:VSSOP-10_3x3mm_P0.5mm; Manufacturer (none) -> Texas Instruments; Part number (none) -> TPS62050DGSR
- U?: footprint (none) -> Package_SO:VSSOP-10_3x3mm_P0.5mm; Manufacturer (none) -> Texas Instruments; Part number (none) -> TPS62056DGSR
Changed lines of the file:
@@
 F 2 "Package_BGA:BGA-256_14.0x14.0mm_Layout16x16_P0.8mm_Ball0.45mm_Pad0.32mm_NSMD" H 13300 1525 50  0001 C CNN
 F 3 "" H 13300 1525 50  0001 C CNN
+F 4 "Lattice" H 13300 1525 50  0001 C CNN "Manufacturer"
+F 5 "iCE40HX8K-CT256" H 13300 1525 50  0001 C CNN "Part number"
 	1    13300 1525
 	1    0    0    -1
@@
 F 0 "U?" H 4450 4850 50  0000 C CNN
 F 1 "TPS62056" H 4450 4775 50  0000 C CNN
-F 2 "" H 4450 4775 50  0001 C CNN
+F 2 "Package_SO:VSSOP-10_3x3mm_P0.5mm" H 4450 4775 50  0001 C CNN
 F 3 "http://www.ti.com/lit/ds/symlink/tps62050.pdf" H 4450 4775 50  0001 C CNN
+F 4 "Texas Instruments" H 4450 4775 50  0001 C CNN "Manufacturer"
+F 5 "TPS62056DGSR " H 4450 4775 50  0001 C CNN "Part number"
 	1    4450 4775
 	1    0    0    -1
@@
 F 0 "U?" H 4450 3275 50  0000 C CNN
 F 1 "TPS62050" H 4450 3200 50  0000 C CNN
-F 2 "" H 4450 3200 50  0001 C CNN
+F 2 "Package_SO:VSSOP-10_3x3mm_P0.5mm" H 4450 3200 50  0001 C CNN
 F 3 "http://www.ti.com/lit/ds/symlink/tps62050.pdf" H 4450 3200 50  0001 C CNN
+F 4 "Texas Instruments " H 4450 3200 50  0001 C CNN "Manufacturer"
+F 5 "TPS62050DGSR" H 4450 3200 50  0001 C CNN "Part number"
 	1    4450 3200
 	1    0    0    -1
@@
 F 0 "U?" H 4450 1525 50  0000 C CNN
 F 1 "TPS62050" H 4450 1450 50  0000 C CNN
-F 2 "" H 4450 1450 50  0001 C CNN
+F 2 "Package_SO:VSSOP-10_3x3mm_P0.5mm" H 4450 1450 50  0001 C CNN
 F 3 "http://www.ti.com/lit/ds/symlink/tps62050.pdf" H 4450 1450 50  0001 C CNN
+F 4 "Texas Instruments " H 4450 1450 50  0001 C CNN "Manufacturer"
+F 5 "TPS62050DGSR" H 4450 1450 50  0001 C CNN "Part number"
 	1    4450 1450
 	1    0    0    -1

Commit message: Footprints.
Parts:
- removed TP? (x9): TestPoint, symbol Connector:TestPoint
- added TP? (x9): TestPoint, TestPoint:TestPoint_Pad_D1.0mm, symbol icenes-library:TestPoint
Changed lines of the file:
@@
 	6050 4875 6100 4875
-$Comp
-L Connector:TestPoint TP?
-U 1 1 5D6A7F85
-P 6100 4800
-F 0 "TP?" H 6175 5000 50  0000 R CNN
-F 1 "TestPoint" H 6042 4917 50  0001 R CNN
-F 2 "" H 6300 4800 50  0001 C CNN
-F 3 "~" H 6300 4800 50  0001 C CNN
-	1    6100 4800
-	1    0    0    -1
-$EndComp
 $Comp
 L icenes-library:R0 R?
@@
 F 6 "RC0805FR-070RL" H 5900 4875 50  0001 C CNN "Part number"
 	1    5900 4875
-	1    0    0    -1
-$EndComp
-$Comp
-L Connector:TestPoint TP?
-U 1 1 5D6A7F78
-P 5700 4800
-F 0 "TP?" H 5775 5000 50  0000 R CNN
-F 1 "TestPoint" H 5642 4917 50  0001 R CNN
-F 2 "" H 5900 4800 50  0001 C CNN
-F 3 "~" H 5900 4800 50  0001 C CNN
-	1    5700 4800
 	1    0    0    -1
 $EndComp
@@
 	5375 5250 5375 5350
 $Comp
-L Connector:TestPoint TP?
-U 1 1 5D446D10
-P 5375 5350
-F 0 "TP?" H 5425 5575 50  0000 R CNN
-F 1 "TestPoint" H 5317 5467 50  0001 R CNN
-F 2 "" H 5575 5350 50  0001 C CNN
-F 3 "~" H 5575 5350 50  0001 C CNN
-	1    5375 5350
-	-1   0    0    1
-$EndComp
-$Comp
 L icenes-library:R1M R?
 U 1 1 5D446D0A
@@
 	6625 3300 6675 3300
 $Comp
-L Connector:TestPoint TP?
-U 1 1 5D56A612
-P 6675 3225
-F 0 "TP?" H 6750 3425 50  0000 R CNN
-F 1 "TestPoint" H 6617 3342 50  0001 R CNN
-F 2 "" H 6875 3225 50  0001 C CNN
-F 3 "~" H 6875 3225 50  0001 C CNN
-	1    6675 3225
-	1    0    0    -1
-$EndComp
-$Comp
 L icenes-library:R0 R?
 U 1 1 5D56A60B
@@
 	0    -1   -1   0
 $EndComp
-$Comp
-L Connector:TestPoint TP?
-U 1 1 5D3F2982
-P 6275 3225
-F 0 "TP?" H 6350 3425 50  0000 R CNN
-F 1 "TestPoint" H 6217 3342 50  0001 R CNN
-F 2 "" H 6475 3225 50  0001 C CNN
-F 3 "~" H 6475 3225 50  0001 C CNN
-	1    6275 3225
-	1    0    0    -1
-$EndComp
 Wire Wire Line
 	4900 4150 5700 4150
@@
 Wire Wire Line
 	5375 3675 5375 3775
-$Comp
-L Connector:TestPoint TP?
-U 1 1 5D3F2979
-P 5375 3775
-F 0 "TP?" H 5425 4000 50  0000 R CNN
-F 1 "TestPoint" H 5317 3892 50  0001 R CNN
-F 2 "" H 5575 3775 50  0001 C CNN
-F 3 "~" H 5575 3775 50  0001 C CNN
-	1    5375 3775
-	-1   0    0    1
-$EndComp
 $Comp
 L icenes-library:R1M R?
@@
 	1    0    0    -1
 $EndComp
-$Comp
-L Connector:TestPoint TP?
-U 1 1 5D508640
-P 6650 1475
-F 0 "TP?" H 6725 1675 50  0000 R CNN
-F 1 "TestPoint" H 6592 1592 50  0001 R CNN
-F 2 "" H 6850 1475 50  0001 C CNN
-F 3 "~" H 6850 1475 50  0001 C CNN
-	1    6650 1475
-	1    0    0    -1
-$EndComp
 Wire Wire Line
 	6900 1450 6900 1550
@@
 Wire Wire Line
 	6250 1475 6250 1550
-$Comp
-L Connector:TestPoint TP?
-U 1 1 5D3CF01A
-P 6250 1475
-F 0 "TP?" H 6325 1675 50  0000 R CNN
-F 1 "TestPoint" H 6192 1592 50  0001 R CNN
-F 2 "" H 6450 1475 50  0001 C CNN
-F 3 "~" H 6450 1475 50  0001 C CNN
-	1    6250 1475
-	1    0    0    -1
-$EndComp
 Wire Wire Line
 	4900 2400 5700 2400
@@
 Wire Wire Line
 	5375 1925 5375 2025
-$Comp
-L Connector:TestPoint TP?
-U 1 1 5D3BB92C
-P 5375 2025
-F 0 "TP?" H 5425 2250 50  0000 R CNN
-F 1 "TestPoint" H 5317 2142 50  0001 R CNN
-F 2 "" H 5575 2025 50  0001 C CNN
-F 3 "~" H 5575 2025 50  0001 C CNN
-	1    5375 2025
-	-1   0    0    1
-$EndComp
 $Comp
 L icenes-library:R1M R?
@@
 	1    0    0    -1
 $EndComp
+$Comp
+L icenes-library:TestPoint TP?
+U 1 1 5D7111E6
+P 6250 1475
+F 0 "TP?" H 6200 1675 50  0000 L CNN
+F 1 "TestPoint" H 6250 1675 50  0001 C CNN
+F 2 "TestPoint:TestPoint_Pad_D1.0mm" H 6450 1475 50  0001 C CNN
+F 3 "~" H 6450 1475 50  0001 C CNN
+	1    6250 1475
+	1    0    0    -1
+$EndComp
+$Comp
+L icenes-library:TestPoint TP?
+U 1 1 5D712B7B
+P 6650 1475
+F 0 "TP?" H 6600 1675 50  0000 L CNN
+F 1 "TestPoint" H 6650 1675 50  0001 C CNN
+F 2 "TestPoint:TestPoint_Pad_D1.0mm" H 6850 1475 50  0001 C CNN
+F 3 "~" H 6850 1475 50  0001 C CNN
+	1    6650 1475
+	1    0    0    -1
+$EndComp
+$Comp
+L icenes-library:TestPoint TP?
+U 1 1 5D724BBE
+P 6275 3225
+F 0 "TP?" H 6225 3425 50  0000 L CNN
+F 1 "TestPoint" H 6275 3425 50  0001 C CNN
+F 2 "TestPoint:TestPoint_Pad_D1.0mm" H 6475 3225 50  0001 C CNN
+F 3 "~" H 6475 3225 50  0001 C CNN
+	1    6275 3225
+	1    0    0    -1
+$EndComp
+$Comp
+L icenes-library:TestPoint TP?
+U 1 1 5D735BB7
+P 6675 3225
+F 0 "TP?" H 6625 3425 50  0000 L CNN
+F 1 "TestPoint" H 6675 3425 50  0001 C CNN
+F 2 "TestPoint:TestPoint_Pad_D1.0mm" H 6875 3225 50  0001 C CNN
+F 3 "~" H 6875 3225 50  0001 C CNN
+	1    6675 3225
+	1    0    0    -1
+$EndComp
+$Comp
+L icenes-library:TestPoint TP?
+U 1 1 5D746D9B
+P 5700 4800
+F 0 "TP?" H 5650 5000 50  0000 L CNN
+F 1 "TestPoint" H 5700 5000 50  0001 C CNN
+F 2 "TestPoint:TestPoint_Pad_D1.0mm" H 5900 4800 50  0001 C CNN
+F 3 "~" H 5900 4800 50  0001 C CNN
+	1    5700 4800
+	1    0    0    -1
+$EndComp
+$Comp
+L icenes-library:TestPoint TP?
+U 1 1 5D758010
+P 6100 4800
+F 0 "TP?" H 6050 5000 50  0000 L CNN
+F 1 "TestPoint" H 6100 5000 50  0001 C CNN
+F 2 "TestPoint:TestPoint_Pad_D1.0mm" H 6300 4800 50  0001 C CNN
+F 3 "~" H 6300 4800 50  0001 C CNN
+	1    6100 4800
+	1    0    0    -1
+$EndComp
+$Comp
+L power:PWR_FLAG #FLG?
+U 1 1 5D7877EF
+P 3250 1550
+F 0 "#FLG?" H 3250 1625 50  0001 C CNN
+F 1 "PWR_FLAG" H 3250 1723 50  0000 C CNN
+F 2 "" H 3250 1550 50  0001 C CNN
+F 3 "~" H 3250 1550 50  0001 C CNN
+	1    3250 1550
+	1    0    0    -1
+$EndComp
+$Comp
+L power:PWR_FLAG #FLG?
+U 1 1 5D7882E7
+P 2425 1750
+F 0 "#FLG?" H 2425 1825 50  0001 C CNN
+F 1 "PWR_FLAG" V 2425 1878 50  0000 L CNN
+F 2 "" H 2425 1750 50  0001 C CNN
+F 3 "~" H 2425 1750 50  0001 C CNN
+	1    2425 1750
+	0    1    1    0
+$EndComp
+$Comp
+L icenes-library:TestPoint TP?
+U 1 1 5D825FFB
+P 5375 5350
+F 0 "TP?" H 5325 5550 50  0000 L CNN
+F 1 "TestPoint" H 5375 5550 50  0001 C CNN
+F 2 "TestPoint:TestPoint_Pad_D1.0mm" H 5575 5350 50  0001 C CNN
+F 3 "~" H 5575 5350 50  0001 C CNN
+	1    5375 5350
+	-1   0    0    1
+$EndComp
+$Comp
+L icenes-library:TestPoint TP?
+U 1 1 5D8379DB
+P 5375 3775
+F 0 "TP?" H 5325 3975 50  0000 L CNN
+F 1 "TestPoint" H 5375 3975 50  0001 C CNN
+F 2 "TestPoint:TestPoint_Pad_D1.0mm" H 5575 3775 50  0001 C CNN
+F 3 "~" H 5575 3775 50  0001 C CNN
+	1    5375 3775
+	-1   0    0    1
+$EndComp
+$Comp
+L icenes-library:TestPoint TP?
+U 1 1 5D848D12
+P 5375 2025
+F 0 "TP?" H 5325 2225 50  0000 L CNN
+F 1 "TestPoint" H 5375 2225 50  0001 C CNN
+F 2 "TestPoint:TestPoint_Pad_D1.0mm" H 5575 2025 50  0001 C CNN
+F 3 "~" H 5575 2025 50  0001 C CNN
+	1    5375 2025
+	-1   0    0    1
+$EndComp
 $EndSCHEMATC

Commit message: Completed USB interface. Clock sources for PAL and NTSC frequencies. Added a 133MHz clock (max input to PLL). Some more stuff.
Parts:
- removed J?: USB_B_Micro, symbol Connector:USB_B_Micro
- removed J?: Barrel_Jack_Switch, symbol Connector:Barrel_Jack_Switch
- added C?: C0.1uF, Capacitor_SMD:C_0603_1608Metric_Pad1.05x0.95mm_HandSolder, symbol icenes-library:C0.1uF
- added C? (x3): C22uF, Capacitor_SMD:C_0603_1608Metric_Pad1.05x0.95mm_HandSolder, symbol icenes-library:C22uF
- added C? (x6): C1uF, Capacitor_SMD:C_0603_1608Metric_Pad1.05x0.95mm_HandSolder, symbol icenes-library:C1uF
- added D?: Green_LED, LED_SMD:LED_0805_2012Metric_Pad1.15x1.40mm_HandSolder, symbol icenes-library:Green_LED
- added FB?: FB600_500mA_0603, Inductor_SMD:L_0603_1608Metric_Pad1.05x0.95mm_HandSolder, symbol icenes-library:FB600_500mA_0603
- added FB? (x3): FB110_4100mA_0603, Inductor_SMD:L_0603_1608Metric_Pad1.05x0.95mm_HandSolder, symbol icenes-library:FB110_4100mA_0603
- added J?: USB_B_Micro, icenes-library:USB_Micro-B, symbol icenes-library:USB_B_Micro
- added J?: Barrel_Jack_Switch, symbol icenes-library:Barrel_Jack_Switch
- added R?: R2.2K, Resistor_SMD:R_0603_1608Metric_Pad1.05x0.95mm_HandSolder, symbol icenes-library:R2.2K
- added TP? (x5): TestPoint, TestPoint:TestPoint_Pad_D1.0mm, symbol icenes-library:TestPoint
Connections:
- net labels added: USB_VBUS
- wire segments 245 -> 309
- no-connect marks 1 -> 2
Other:
- moved on the sheet: C?, D?, U?A

Commit message: Added missing footprints.
Parts:
- J?: footprint (none) -> icenes-library:BarrelJack_Horizontal; Maufacturer (none) -> Kobiconn; Part number (none) -> 163-179PH-EX
Changed lines of the file:
@@
 F 0 "J?" H 2132 1967 50  0000 C CNN
 F 1 "Barrel_Jack_Switch" H 2132 1876 50  0000 C CNN
-F 2 "" H 2125 1610 50  0001 C CNN
-F 3 "~" H 2125 1610 50  0001 C CNN
+F 2 "icenes-library:BarrelJack_Horizontal" H 2125 1610 50  0001 C CNN
+F 3 "https://www.mouser.se/datasheet/2/253/KC-301287-1177723.pdf" H 2125 1610 50  0001 C CNN
+F 4 "Kobiconn" H 2075 1650 50  0001 C CNN "Maufacturer"
+F 5 "163-179PH-EX" H 2075 1650 50  0001 C CNN "Part number"
 	1    2075 1650
 	1    0    0    -1

Commit message: Minor fixes.
Parts:
- gave numbers to parts that had none: 73

Commit message: Fixed all ECR warnings.
Parts:
- added C16, C20: C0.1uF, Capacitor_SMD:C_0603_1608Metric_Pad1.05x0.95mm_HandSolder, symbol icenes-library:C0.1uF
- added R12: R0, Resistor_SMD:R_0805_2012Metric_Pad1.15x1.40mm_HandSolder, symbol icenes-library:R0
- added TP12, TP13: TestPoint, TestPoint:TestPoint_Pad_D1.0mm, symbol icenes-library:TestPoint
- renumbered C16 to C17, C17 to C18, C18 to C19, C19 to C21, C20 to C22, C21 to C23, C22 to C24, C23 to C25, C24 to C26, C25 to C27, C26 to C28, C27 to C29, C28 to C30, C29 to C31, C30 to C32, C31 to C33, C32 to C34, C33 to C35, TP12 to TP14, TP13 to TP15, TP14 to TP16
Connections:
- net +3V3: now also R12.1, TP12.1
- net +3V3_FTDI: now also C16.1, C20.1, R12.2, TP13.1
- net GND: now also C16.2, C20.2; no longer U1.2 (LBO), U2.2 (LBO), U3.2 (LBO)
- no-connect marks 2 -> 5
Other:
- moved on the sheet: C10, C4, C7, FB2, L3, R4, R9, TP14, TP5, TP6, TP7, U3
