File: hw/icenes-io1.sch (KiCad schematic (older format))
At the start: 49 parts, among them J3 Conn_02x11_Odd_Even, U4 iCE40HX8K-CT256, U8 SN74LVC1404, U9 SN74LVC1404, Y1 21.47727MHz, Y2 26.601712MHz

Commit message: Fixed all ECR warnings.
Changed lines of the file:
@@
 	2700 2000 2700 1900
 $Comp
-L power:+3V3 #PWR052
+L power:+3V3 #PWR058
 U 1 1 5D2FE82F
 P 950 1800
-F 0 "#PWR052" H 950 1650 50  0001 C CNN
+F 0 "#PWR058" H 950 1650 50  0001 C CNN
 F 1 "+3V3" H 965 1973 50  0000 C CNN
 F 2 "" H 950 1800 50  0001 C CNN
@@
 $EndComp
 $Comp
-L power:GND #PWR057
+L power:GND #PWR063
 U 1 1 5D3005C9
 P 2300 2350
-F 0 "#PWR057" H 2300 2100 50  0001 C CNN
+F 0 "#PWR063" H 2300 2100 50  0001 C CNN
 F 1 "GND" H 2305 2177 50  0000 C CNN
 F 2 "" H 2300 2350 50  0001 C CNN
@@
 	9700 2000 9700 1900
 $Comp
-L power:+3V3 #PWR065
+L power:+3V3 #PWR071
 U 1 1 5D30FC3B
 P 7950 1800
-F 0 "#PWR065" H 7950 1650 50  0001 C CNN
+F 0 "#PWR071" H 7950 1650 50  0001 C CNN
 F 1 "+3V3" H 7965 1973 50  0000 C CNN
 F 2 "" H 7950 1800 50  0001 C CNN
@@
 $EndComp
 $Comp
-L power:GND #PWR070
+L power:GND #PWR076
 U 1 1 5D30FC41
 P 9300 2350
-F 0 "#PWR070" H 9300 2100 50  0001 C CNN
+F 0 "#PWR076" H 9300 2100 50  0001 C CNN
 F 1 "GND" H 9305 2177 50  0000 C CNN
 F 2 "" H 9300 2350 50  0001 C CNN
@@
 $EndComp
 $Comp
-L power:+1V2 #PWR054
+L power:+1V2 #PWR060
 U 1 1 5D312958
 P 1850 3000
-F 0 "#PWR054" H 1850 2850 50  0001 C CNN
+F 0 "#PWR060" H 1850 2850 50  0001 C CNN
 F 1 "+1V2" H 1865 3173 50  0000 C CNN
 F 2 "" H 1850 3000 50  0001 C CNN
@@
 $EndComp
 $Comp
-L power:GND #PWR073
+L power:GND #PWR079
 U 1 1 5D436A19
 P 11275 7625
-F 0 "#PWR073" H 11275 7375 50  0001 C CNN
+F 0 "#PWR079" H 11275 7375 50  0001 C CNN
 F 1 "GND" H 11280 7452 50  0000 C CNN
 F 2 "" H 11275 7625 50  0001 C CNN
@@
 $EndComp
 $Comp
-L power:GND #PWR079
+L power:GND #PWR085
 U 1 1 5D4BD4BD
 P 13150 7625
-F 0 "#PWR079" H 13150 7375 50  0001 C CNN
+F 0 "#PWR085" H 13150 7375 50  0001 C CNN
 F 1 "GND" H 13155 7452 50  0000 C CNN
 F 2 "" H 13150 7625 50  0001 C CNN
@@
 $EndComp
 $Comp
-L power:GND #PWR080
+L power:GND #PWR086
 U 1 1 5D4C38DD
 P 13525 7625
-F 0 "#PWR080" H 13525 7375 50  0001 C CNN
+F 0 "#PWR086" H 13525 7375 50  0001 C CNN
 F 1 "GND" H 13530 7452 50  0000 C CNN
 F 2 "" H 13525 7625 50  0001 C CNN
@@
 $EndComp
 $Comp
-L power:GND #PWR081
+L power:GND #PWR087
 U 1 1 5D4C9724
 P 13900 7625
-F 0 "#PWR081" H 13900 7375 50  0001 C CNN
+F 0 "#PWR087" H 13900 7375 50  0001 C CNN
 F 1 "GND" H 13905 7452 50  0000 C CNN
 F 2 "" H 13900 7625 50  0001 C CNN
@@
 	9225 8450 9225 8500
 $Comp
-L power:GND #PWR069
+L power:GND #PWR075
 U 1 1 5D6F756D
 P 9225 8500
-F 0 "#PWR069" H 9225 8250 50  0001 C CNN
+F 0 "#PWR075" H 9225 8250 50  0001 C CNN
 F 1 "GND" H 9230 8327 50  0000 C CNN
 F 2 "" H 9225 8500 50  0001 C CNN
@@
 $EndComp
 $Comp
-L power:GND #PWR074
+L power:GND #PWR080
 U 1 1 5D6F55B4
 P 11275 8600
-F 0 "#PWR074" H 11275 8350 50  0001 C CNN
+F 0 "#PWR080" H 11275 8350 50  0001 C CNN
 F 1 "GND" H 11280 8427 50  0000 C CNN
 F 2 "" H 11275 8600 50  0001 C CNN
@@
 $EndComp
 $Comp
-L power:+3V3 #PWR068
+L power:+3V3 #PWR074
 U 1 1 5D6F4A08
 P 9225 8100
-F 0 "#PWR068" H 9225 7950 50  0001 C CNN
+F 0 "#PWR074" H 9225 7950 50  0001 C CNN
 F 1 "+3V3" H 9240 8273 50  0000 C CNN
 F 2 "" H 9225 8100 50  0001 C CNN
@@
 	9700 8450 9700 8500
 $Comp
-L power:GND #PWR072
+L power:GND #PWR078
 U 1 1 5D758924
 P 9700 8500
-F 0 "#PWR072" H 9700 8250 50  0001 C CNN
+F 0 "#PWR078" H 9700 8250 50  0001 C CNN
 F 1 "GND" H 9705 8327 50  0000 C CNN
 F 2 "" H 9700 8500 50  0001 C CNN
@@
 	8750 8450 8750 8500
 $Comp
-L power:GND #PWR067
+L power:GND #PWR073
 U 1 1 5D763419
 P 8750 8500
-F 0 "#PWR067" H 8750 8250 50  0001 C CNN
+F 0 "#PWR073" H 8750 8250 50  0001 C CNN
 F 1 "GND" H 8755 8327 50  0000 C CNN
 F 2 "" H 8750 8500 50  0001 C CNN
@@
 $EndComp
 $Comp
-L power:+1V2 #PWR071
+L power:+1V2 #PWR077
 U 1 1 5D76E658
 P 9700 8100
-F 0 "#PWR071" H 9700 7950 50  0001 C CNN
+F 0 "#PWR077" H 9700 7950 50  0001 C CNN
 F 1 "+1V2" H 9715 8273 50  0000 C CNN
 F 2 "" H 9700 8100 50  0001 C CNN
@@
 $EndComp
 $Comp
-L power:+5V #PWR066
+L power:+5V #PWR072
 U 1 1 5D76F52B
 P 8750 8100
-F 0 "#PWR066" H 8750 7950 50  0001 C CNN
+F 0 "#PWR072" H 8750 7950 50  0001 C CNN
 F 1 "+5V" H 8765 8273 50  0000 C CNN
 F 2 "" H 8750 8100 50  0001 C CNN
@@
 $EndComp
 $Comp
-L power:GND #PWR078
+L power:GND #PWR084
 U 1 1 5D4B6CF0
 P 12775 7625
-F 0 "#PWR078" H 12775 7375 50  0001 C CNN
+F 0 "#PWR084" H 12775 7375 50  0001 C CNN
 F 1 "GND" H 12780 7452 50  0000 C CNN
 F 2 "" H 12775 7625 50  0001 C CNN
@@
 $EndComp
 $Comp
-L power:GND #PWR077
+L power:GND #PWR083
 U 1 1 5D4B0BFC
 P 12400 7625
-F 0 "#PWR077" H 12400 7375 50  0001 C CNN
+F 0 "#PWR083" H 12400 7375 50  0001 C CNN
 F 1 "GND" H 12405 7452 50  0000 C CNN
 F 2 "" H 12400 7625 50  0001 C CNN
@@
 $EndComp
 $Comp
-L power:GND #PWR076
+L power:GND #PWR082
 U 1 1 5D4AAC07
 P 12025 7625
-F 0 "#PWR076" H 12025 7375 50  0001 C CNN
+F 0 "#PWR082" H 12025 7375 50  0001 C CNN
 F 1 "GND" H 12030 7452 50  0000 C CNN
 F 2 "" H 12025 7625 50  0001 C CNN
@@
 $EndComp
 $Comp
-L power:GND #PWR075
+L power:GND #PWR081
 U 1 1 5D49EA59
 P 11650 7625
-F 0 "#PWR075" H 11650 7375 50  0001 C CNN
+F 0 "#PWR081" H 11650 7375 50  0001 C CNN
 F 1 "GND" H 11655 7452 50  0000 C CNN
 F 2 "" H 11650 7625 50  0001 C CNN
@@
 $EndComp
 $Comp
-L power:+3V3 #PWR058
+L power:+3V3 #PWR064
 U 1 1 5D64E041
 P 3300 8100
-F 0 "#PWR058" H 3300 7950 50  0001 C CNN
+F 0 "#PWR064" H 3300 7950 50  0001 C CNN
 F 1 "+3V3" H 3315 8273 50  0000 C CNN
 F 2 "" H 3300 8100 50  0001 C CNN
@@
 $EndComp
 $Comp
-L power:GND #PWR059
+L power:GND #PWR065
 U 1 1 5D6510AE
 P 3300 8450
-F 0 "#PWR059" H 3300 8200 50  0001 C CNN
+F 0 "#PWR065" H 3300 8200 50  0001 C CNN
 F 1 "GND" H 3305 8277 50  0000 C CNN
 F 2 "" H 3300 8450 50  0001 C CNN
@@
 	1950 9775 1950 9750
 $Comp
-L power:GND #PWR056
+L power:GND #PWR062
 U 1 1 5D65DE4D
 P 2075 9100
-F 0 "#PWR056" H 2075 8850 50  0001 C CNN
+F 0 "#PWR062" H 2075 8850 50  0001 C CNN
 F 1 "GND" H 2080 8927 50  0000 C CNN
 F 2 "" H 2075 9100 50  0001 C CNN
@@
 $EndComp
 $Comp
-L power:GND #PWR055
+L power:GND #PWR061
 U 1 1 5D64CDC5
 P 1950 9775
-F 0 "#PWR055" H 1950 9525 50  0001 C CNN
+F 0 "#PWR061" H 1950 9525 50  0001 C CNN
 F 1 "GND" H 1955 9602 50  0000 C CNN
 F 2 "" H 1950 9775 50  0001 C CNN
@@
 $EndComp
 $Comp
-L power:GND #PWR053
+L power:GND #PWR059
 U 1 1 5D64BB5A
 P 1050 9775
-F 0 "#PWR053" H 1050 9525 50  0001 C CNN
+F 0 "#PWR059" H 1050 9525 50  0001 C CNN
 F 1 "GND" H 1055 9602 50  0000 C CNN
 F 2 "" H 1050 9775 50  0001 C CNN
@@
 $EndComp
 $Comp
-L power:+3V3 #PWR063
+L power:+3V3 #PWR069
 U 1 1 5DB221B3
 P 7075 8100
-F 0 "#PWR063" H 7075 7950 50  0001 C CNN
+F 0 "#PWR069" H 7075 7950 50  0001 C CNN
 F 1 "+3V3" H 7090 8273 50  0000 C CNN
 F 2 "" H 7075 8100 50  0001 C CNN
@@
 $EndComp
 $Comp
-L power:GND #PWR064
+L power:GND #PWR070
 U 1 1 5DB221C2
 P 7075 8450
-F 0 "#PWR064" H 7075 8200 50  0001 C CNN
+F 0 "#PWR070" H 7075 8200 50  0001 C CNN
 F 1 "GND" H 7080 8277 50  0000 C CNN
 F 2 "" H 7075 8450 50  0001 C CNN
@@
 	5725 9775 5725 9750
 $Comp
-L power:GND #PWR062
+L power:GND #PWR068
 U 1 1 5DB221DA
 P 5850 9100
-F 0 "#PWR062" H 5850 8850 50  0001 C CNN
+F 0 "#PWR068" H 5850 8850 50  0001 C CNN
 F 1 "GND" H 5855 8927 50  0000 C CNN
 F 2 "" H 5850 9100 50  0001 C CNN
@@
 $EndComp
 $Comp
-L power:GND #PWR061
+L power:GND #PWR067
 U 1 1 5DB221E0
 P 5725 9775
-F 0 "#PWR061" H 5725 9525 50  0001 C CNN
+F 0 "#PWR067" H 5725 9525 50  0001 C CNN
 F 1 "GND" H 5730 9602 50  0000 C CNN
 F 2 "" H 5725 9775 50  0001 C CNN
@@
 $EndComp
 $Comp
-L power:GND #PWR060
+L power:GND #PWR066
 U 1 1 5DB221E6
 P 4825 9775
-F 0 "#PWR060" H 4825 9525 50  0001 C CNN
+F 0 "#PWR066" H 4825 9525 50  0001 C CNN
 F 1 "GND" H 4830 9602 50  0000 C CNN
 F 2 "" H 4825 9775 50  0001 C CNN
@@
 Wire Wire Line
 	9475 6800 9850 6800
+$Comp
+L power:PWR_FLAG #FLG?
+U 1 1 5E05F6AC
+P 2300 3550
+AR Path="/5E05F6AC" Ref="#FLG?"  Part="1"
+AR Path="/5D1BB1FB/5E05F6AC" Ref="#FLG0103"  Part="1"
+F 0 "#FLG0103" H 2300 3625 50  0001 C CNN
+F 1 "PWR_FLAG" H 2300 3723 50  0000 C CNN
+F 2 "" H 2300 3550 50  0001 C CNN
+F 3 "~" H 2300 3550 50  0001 C CNN
+	1    2300 3550
+	-1   0    0    1
+$EndComp
+Wire Wire Line
+	2300 3550 2300 3500
 $EndSCHEMATC
