File: hw/icenes-io1.sch (KiCad schematic (older format))
At the start: 45 parts, among them U4 iCE40HX8K-CT256, U8 SN74LVC1404, U9 SN74LVC1404, Y1 21.47727MHz, Y2 26.601712MHz

Commit message: Layout.
Connections:
- net GPIO_G14 is gone; now on net CPU_DATA_DIR: U4.G14 (IO1_37)
- net GPIO_H11 is gone; now on net ~ICE_PPU_RD: U4.H11 (GBIN3/IO1_27)
- net GPIO_H12 is gone; now on net ~ICE_ROMSEL: U4.H12 (IO1_31)
- net GPIO_J11 is gone; now on net ICE_SYSTEM_CLK: U4.J11 (IO1_15)
- net GPIO_J12 is gone; now on net ~MISC_OE1: U4.J12 (IO1_23)
- net GPIO_J13 is gone; now on net MISC_DIR1: U4.J13 (IO1_24)
- net ICE_M2 is gone; now on net ICE_CICtoMB: U4.F12 (IO1_43)
- net CPU_ADDR_DIR: now also U4.B4 (IO0_41); no longer U4.D7 (IO0_35)
- net CPU_DATA_DIR: no longer U4.F14 (IO1_42)
- net ICE_CICtoMB: no longer U4.E13 (IO1_50)
- net ICE_CICtoPak: now also U4.G12 (IO1_41); no longer U4.G13 (IO1_39)
- net ICE_CIRAM_A10: now also U4.E13 (IO1_50); no longer U4.F15 (IO1_36)
- net ICE_CLK_26.601712MHz: no longer U4.F7 (GBIN0/IO0_26)
- net ICE_CPU_A0: now also U4.B3 (IO0_47); no longer U4.B8 (IO0_29)
- net ICE_CPU_A1: now also U4.C3 (IO0_51); no longer U4.B7 (IO0_32)
- net ICE_CPU_A10: now also U4.D7 (IO0_35); no longer U4.B5 (IO0_39)
- net ICE_CPU_A11: now also U4.D6 (IO0_37); no longer U4.C3 (IO0_51)
- net ICE_CPU_A12: now also U4.E6 (IO0_40); no longer U4.B4 (IO0_41)
- net ICE_CPU_A13: now also U4.D5 (IO0_43); no longer U4.A2 (IO0_42)
- net ICE_CPU_A14: now also U4.E5 (IO0_49); no longer U4.D3 (IO0_50)
- net ICE_CPU_A2: now also U4.A2 (IO0_42); no longer U4.D6 (IO0_37)
- net ICE_CPU_A3: now also U4.A1 (IO0_44); no longer U4.A7 (IO0_30)
- net ICE_CPU_A4: now also U4.D10 (IO0_19); no longer U4.B6 (IO0_33)
- net ICE_CPU_A5: now also U4.E10 (IO0_10); no longer U4.C5 (IO0_45)
- net ICE_CPU_A6: now also U4.D9 (IO0_22); no longer U4.C4 (IO0_46)
- net ICE_CPU_A7: now also U4.E9 (IO0_21); no longer U4.A6 (IO0_36)
- net ICE_CPU_A8: now also U4.F9 (IO0_24); no longer U4.B3 (IO0_47)
- net ICE_CPU_A9: now also U4.D8 (IO0_28); no longer U4.A5 (IO0_38)
- net ICE_CPU_D0: now also U4.F15 (IO1_36); no longer U4.F16 (IO1_34)
- net ICE_CPU_D1: now also U4.F14 (IO1_42); no longer U4.E16 (IO1_38)
- net ICE_CPU_D2: now also U4.E16 (IO1_38); no longer U4.D16 (IO1_40)
- net ICE_CPU_D4: now also U4.D15 (IO1_44); no longer U4.D14 (IO1_51)
- net ICE_CPU_D5: now also U4.D14 (IO1_51); no longer U4.D15 (IO1_44)
- net ICE_CPU_RW: now also U4.D4 (IO0_48); no longer U4.A1 (IO0_44)
- net ICE_PPU_A0: now also U4.B11 (IO0_15); no longer U4.B12 (IO0_13)
- net ICE_PPU_A1: now also U4.A11 (IO0_18); no longer U4.B11 (IO0_15)
- net ICE_PPU_A10: now also U4.B7 (IO0_32); no longer U4.C9 (IO0_20)
- net ICE_PPU_A11: now also U4.C7 (IO0_31); no longer U4.B9 (IO0_27)
- net ICE_PPU_A12: now also U4.A6 (IO0_36); no longer U4.D9 (IO0_22)
- net ICE_PPU_A13: now also U4.C6 (IO0_34); no longer U4.A9 (IO0_23)
- net ICE_PPU_A2: now also U4.C10 (IO0_16); no longer U4.E9 (IO0_21)
- net ICE_PPU_A3: now also U4.B10 (IO0_14); no longer U4.D8 (IO0_28)
- net ICE_PPU_A4: now also U4.A10 (IO0_17); no longer U4.E6 (IO0_40)
- net ICE_PPU_A5: now also U4.B9 (IO0_27); no longer U4.C11 (IO0_11)
- net ICE_PPU_A6: now also U4.A9 (IO0_23); no longer U4.C10 (IO0_16)
- net ICE_PPU_A7: now also U4.B8 (IO0_29); no longer U4.A11 (IO0_18)
- net ICE_PPU_A8: now also U4.C8 (GBIN1/IO0_25); no longer U4.B10 (IO0_14)
- net ICE_PPU_A9: now also U4.A7 (IO0_30); no longer U4.A10 (IO0_17)
- net ICE_PPU_D0: now also U4.A16 (IO0_07); no longer U4.B15 (IO0_01)
- net ICE_PPU_D1: now also U4.B15 (IO0_01); no longer U4.C14 (IO0_00)
- net ICE_PPU_D2: now also U4.A15 (IO0_08); no longer U4.G11 (IO1_35)
- net ICE_PPU_D3: now also U4.C14 (IO0_00); no longer U4.G10 (IO1_33)
- net ICE_PPU_D4: now also U4.C13 (IO0_06); no longer U4.E10 (IO0_10)
- net ICE_PPU_D5: now also U4.B13 (IO0_09); no longer U4.F9 (IO0_24)
- net ICE_PPU_D6: now also U4.C12 (IO0_04); no longer U4.A16 (IO0_07)
- net ICE_PPU_D7: now also U4.B12 (IO0_13); no longer U4.A15 (IO0_08)
- net ICE_SYSTEM_CLK: no longer U4.G12 (IO1_41)
- net LED0: now also U4.G15 (IO1_32); no longer U4.F11 (IO1_45)
- net LED1: now also U4.D16 (IO1_40); no longer U4.D13 (IO0_02)
- net LED2: now also U4.B14 (IO0_03); no longer U4.E11 (IO0_05)
- net LED3: now also U4.E11 (IO0_05); no longer U4.D11 (IO0_12)
- net LED4: now also U4.G10 (IO1_33); no longer U4.D10 (IO0_19)
- net LED5: now also U4.C9 (IO0_20); no longer U4.E5 (IO0_49)
- net LED6: now also U4.B6 (IO0_33); no longer U4.D5 (IO0_43)
- net LED7: now also U4.C5 (IO0_45); no longer U4.D4 (IO0_48)
- net MISC_DIR1: no longer U4.M16 (IO1_12)
- net MISC_DIR2: now also U4.G16 (IO1_30); no longer U4.J16 (IO1_25)
- net PPU_ADDR_DIR: now also U4.D11 (IO0_12); no longer U4.C13 (IO0_06)
- net PPU_DATA_DIR: now also U4.F11 (IO1_45); no longer U4.B13 (IO0_09)
- net ~CPU_ADDR_OE: now also U4.C4 (IO0_46); no longer U4.C6 (IO0_34)
- net ~CPU_DATA_OE: now also U4.F16 (IO1_34); no longer U4.G16 (IO1_30)
- net ~ICE_CIC_RST: now also U4.G13 (IO1_39); no longer U4.F13 (IO1_48)
- net ~ICE_CIRAM_CE: now also U4.G11 (IO1_35); no longer U4.G15 (IO1_32)
- net ~ICE_IRQ: now also U4.F13 (IO1_48); no longer U4.H14 (IO1_29)
- net ~ICE_PPU_A13: now also U4.A5 (IO0_38); no longer U4.C8 (GBIN1/IO0_25)
- net ~ICE_PPU_RD: no longer U4.K15 (IO1_20)
- net ~ICE_PPU_WR: now also U4.B5 (IO0_39); no longer U4.C7 (IO0_31)
- net ~ICE_ROMSEL: no longer U4.K16 (IO1_21)
- net ~MISC_OE1: no longer U4.L16 (IO1_16)
- net ~MISC_OE2: now also U4.H14 (IO1_29); no longer U4.J15 (IO1_19)
- net ~PPU_ADDR_OE: now also U4.C11 (IO0_11); no longer U4.C12 (IO0_04)
- net ~PPU_DATA_OE: now also U4.D13 (IO0_02); no longer U4.B14 (IO0_03)
- new net GPIO_J15: U4.J15 (IO1_19)
- new net GPIO_J16: U4.J16 (IO1_25)
- new net GPIO_K15: U4.K15 (IO1_20)
- new net GPIO_K16: U4.K16 (IO1_21)
- new net GPIO_L16: U4.L16 (IO1_16)
- new net GPIO_M16: U4.M16 (IO1_12)
- no-connect marks 4 -> 6
Other:
- moved on the sheet: TP15

Commit message: Layout.
Connections:
- net ICE_PPU_A10: now also U4.A7 (IO0_30); no longer U4.B7 (IO0_32)
- net ICE_PPU_A11: now also U4.B7 (IO0_32); no longer U4.C7 (IO0_31)
- net ICE_PPU_A12: now also U4.C8 (GBIN1/IO0_25); no longer U4.A6 (IO0_36)
- net ICE_PPU_A13: now also U4.B8 (IO0_29); no longer U4.C6 (IO0_34)
- net ICE_PPU_A7: now also U4.C6 (IO0_34); no longer U4.B8 (IO0_29)
- net ICE_PPU_A8: now also U4.A6 (IO0_36); no longer U4.C8 (GBIN1/IO0_25)
- net ICE_PPU_A9: now also U4.C7 (IO0_31); no longer U4.A7 (IO0_30)
Changed lines of the file:
@@
 Wire Wire Line
 	2800 3200 2850 3200
+Text GLabel 2700 6800 0    50   Output ~ 0
+ICE_PPU_A12
+Text GLabel 4300 4900 2    50   Output ~ 0
+ICE_PPU_A11
 Text GLabel 4300 5300 2    50   Output ~ 0
-ICE_PPU_A12
-Text GLabel 4300 4800 2    50   Output ~ 0
-ICE_PPU_A11
-Text GLabel 4300 4700 2    50   Output ~ 0
-ICE_PPU_A9
-Text GLabel 2700 6800 0    50   Output ~ 0
 ICE_PPU_A8
-Text GLabel 4300 4600 2    50   Output ~ 0
+Text GLabel 4300 5100 2    50   Output ~ 0
 ICE_PPU_A7
 Text GLabel 4300 4200 2    50   Output ~ 0
@@
 	4150 3300 4300 3300
 Wire Wire Line
+	4150 5300 4300 5300
+Wire Wire Line
+	4150 4200 4300 4200
+Wire Wire Line
+	4150 5100 4300 5100
+Wire Wire Line
+	4150 3600 4300 3600
+Wire Wire Line
+	4150 4900 4300 4900
+Wire Wire Line
 	2850 6800 2700 6800
-Wire Wire Line
-	4150 4200 4300 4200
-Wire Wire Line
-	4150 4700 4300 4700
-Wire Wire Line
-	4150 4600 4300 4600
-Wire Wire Line
-	4150 3600 4300 3600
-Wire Wire Line
-	4150 4800 4300 4800
-Wire Wire Line
-	4150 5300 4300 5300
 Text GLabel 4300 6400 2    50   Output ~ 0
 ICE_CPU_A0
@@
 Text GLabel 4300 4000 2    50   Output ~ 0
 ICE_CPU_A7
-Text GLabel 4300 4300 2    50   Output ~ 0
-ICE_CPU_A8
 Text GLabel 4300 4500 2    50   Output ~ 0
 ICE_CPU_A9
 Text GLabel 4300 5200 2    50   Output ~ 0
 ICE_CPU_A10
-Text GLabel 4300 5400 2    50   Output ~ 0
-ICE_CPU_A11
 Text GLabel 4300 5700 2    50   Output ~ 0
 ICE_CPU_A12
@@
 	4150 4000 4300 4000
 Wire Wire Line
-	4150 4300 4300 4300
-Wire Wire Line
 	4150 4500 4300 4500
 Wire Wire Line
 	4150 5200 4300 5200
-Wire Wire Line
-	4150 5400 4300 5400
 Wire Wire Line
 	4150 5700 4300 5700
@@
 NoConn ~ 4150 6700
 Wire Wire Line
-	4150 4900 4300 4900
-Text GLabel 4300 4900 2    50   Output ~ 0
+	4150 4700 4300 4700
+Text GLabel 4300 4700 2    50   Output ~ 0
 ICE_PPU_A10
 Wire Wire Line
@@
 	4150 6600 4300 6600
 Wire Wire Line
-	4150 5100 4300 5100
-Text GLabel 4300 5100 2    50   Output ~ 0
+	4150 4600 4300 4600
+Text GLabel 4300 4600 2    50   Output ~ 0
 ICE_PPU_A13
+Wire Wire Line
+	4150 4300 4300 4300
+Text GLabel 4300 4300 2    50   Output ~ 0
+ICE_CPU_A8
+Wire Wire Line
+	4150 4800 4300 4800
+Text GLabel 4300 4800 2    50   Output ~ 0
+ICE_PPU_A9
+Wire Wire Line
+	4150 5400 4300 5400
+Text GLabel 4300 5400 2    50   Output ~ 0
+ICE_CPU_A11
 $EndSCHEMATC
