File: hw/icenes-usb-flash.sch (KiCad schematic (older format))
At the start: 30 parts

Commit message: Added voltage generators for 3.3V, 1.2V and 5V. Added more info and footprints to some components. Connected signals to the NES connector to banks 0 and 1.
Parts:
- removed R?: R12K@1%, symbol icenes-library:R12K@1%
- added R?: R12K, Resistor_SMD:R_0603_1608Metric_Pad1.05x0.95mm_HandSolder, symbol icenes-library:R12K
- C?: footprint (none) -> Capacitor_SMD:C_0603_1608Metric_Pad1.05x0.95mm_HandSolder; Manufacturer (none) -> Murata; Part number (none) -> GRM188R61A106KE69D
- C? (x12): footprint (none) -> Capacitor_SMD:C_0603_1608Metric_Pad1.05x0.95mm_HandSolder; Manufacturer (none) -> Wurth; Part number (none) -> 885012206020
- C? (x2): footprint (none) -> Capacitor_SMD:C_0603_1608Metric_Pad1.05x0.95mm_HandSolder; Manufacturer (none) -> Taiyo Yuden; Part number (none) -> LMK107BJ475KA-T
- R? (x2): footprint (none) -> Resistor_SMD:R_0603_1608Metric_Pad1.05x0.95mm_HandSolder; Manufacturer (none) -> Yageo; Part number (none) -> RC0603FR-072K2L
- R? (x7): footprint (none) -> Resistor_SMD:R_0603_1608Metric_Pad1.05x0.95mm_HandSolder; Manufacturer (none) -> Yageo; Part number (none) -> RC0603FR-0710KL

Commit message: GPIO headers for banks 2 and 3.
Parts:
- added R?: R0, Resistor_SMD:R_0805_2012Metric_Pad1.15x1.40mm_HandSolder, symbol icenes-library:R0
- added TP? (x2): TestPoint, symbol Connector:TestPoint
Connections:
- wire segments 174 -> 182
Changed lines of the file:
@@
 	1    0    0    -1
 $EndComp
+$Comp
+L icenes-library:+3V3_FTDI #PWR?
+U 1 1 5D3F4BF6
+P 2175 1225
+F 0 "#PWR?" H 2175 1225 50  0001 C CNN
+F 1 "+3V3_FTDI" H 2160 1248 50  0000 C CNN
+F 2 "" H 2175 1225 50  0001 C CNN
+F 3 "" H 2175 1225 50  0001 C CNN
+	1    2175 1225
+	1    0    0    -1
+$EndComp
+Wire Wire Line
+	1825 1425 1825 1500
+Wire Wire Line
+	1425 1500 1475 1500
+Wire Wire Line
+	1425 1425 1425 1500
+Wire Wire Line
+	1775 1500 1825 1500
+$Comp
+L Connector:TestPoint TP?
+U 1 1 5D3FF502
+P 1825 1425
+AR Path="/5D3FF502" Ref="TP?"  Part="1"
+AR Path="/5D1BAC88/5D3FF502" Ref="TP?"  Part="1"
+F 0 "TP?" H 1900 1625 50  0000 R CNN
+F 1 "TestPoint" H 1767 1542 50  0001 R CNN
+F 2 "" H 2025 1425 50  0001 C CNN
+F 3 "~" H 2025 1425 50  0001 C CNN
+	1    1825 1425
+	1    0    0    -1
+$EndComp
+$Comp
+L icenes-library:R0 R?
+U 1 1 5D3FF50B
+P 1625 1500
+AR Path="/5D3FF50B" Ref="R?"  Part="1"
+AR Path="/5D1BAC88/5D3FF50B" Ref="R?"  Part="1"
+F 0 "R?" H 1625 1707 50  0000 C CNN
+F 1 "R0" H 1625 1400 50  0001 C CNN
+F 2 "Resistor_SMD:R_0805_2012Metric_Pad1.15x1.40mm_HandSolder" V 1625 1500 50  0001 C CNN
+F 3 "" V 1625 1500 50  0001 C CNN
+F 4 "0" H 1625 1616 50  0000 C CNN "Resistance"
+F 5 "Yageo" H 1625 1500 50  0001 C CNN "Manufacturer"
+F 6 "RC0805FR-070RL" H 1625 1500 50  0001 C CNN "Part number"
+	1    1625 1500
+	1    0    0    -1
+$EndComp
+$Comp
+L Connector:TestPoint TP?
+U 1 1 5D3FF511
+P 1425 1425
+AR Path="/5D3FF511" Ref="TP?"  Part="1"
+AR Path="/5D1BAC88/5D3FF511" Ref="TP?"  Part="1"
+F 0 "TP?" H 1500 1625 50  0000 R CNN
+F 1 "TestPoint" H 1367 1542 50  0001 R CNN
+F 2 "" H 1625 1425 50  0001 C CNN
+F 3 "~" H 1625 1425 50  0001 C CNN
+	1    1425 1425
+	1    0    0    -1
+$EndComp
+Connection ~ 1425 1500
+Wire Wire Line
+	1825 1500 2175 1500
+Wire Wire Line
+	2175 1500 2175 1375
+Connection ~ 1825 1500
+$Comp
+L power:+3V3 #PWR?
+U 1 1 5D3FF4F2
+P 1075 1375
+AR Path="/5D3FF4F2" Ref="#PWR?"  Part="1"
+AR Path="/5D1BAC88/5D3FF4F2" Ref="#PWR?"  Part="1"
+F 0 "#PWR?" H 1075 1225 50  0001 C CNN
+F 1 "+3V3" H 1090 1548 50  0000 C CNN
+F 2 "" H 1075 1375 50  0001 C CNN
+F 3 "" H 1075 1375 50  0001 C CNN
+	1    1075 1375
+	1    0    0    -1
+$EndComp
+Wire Wire Line
+	1075 1500 1075 1375
+Wire Wire Line
+	1075 1500 1425 1500
 $EndSCHEMATC

Commit message: Footprints.
Parts:
- removed U?: FT2232H, symbol Interface_USB:FT2232H
- added U?: FT2232H, Package_QFP:LQFP-64_10x10mm_P0.5mm, symbol icenes-library:FT2232H
- U?: footprint (none) -> Package_SO:SOIC-8_3.9x4.9mm_P1.27mm; Manufacturer (none) -> Microchip; Part number (none) -> 93LC56C-I/SN
- U?: footprint (none) -> Package_SO:SOIC-8_3.9x4.9mm_P1.27mm; Manufacturer (none) -> Adesto Technologies; Part number (none) -> AT25SF041-SSHD-B
- U?: Manufacturer (none) -> Lattice; Part number (none) -> iCE40HX8K-CT256
- X?: footprint (none) -> Crystal:Crystal_SMD_2520-4Pin_2.5x2.0mm; Manufacturer (none) -> Microchip; Part number (none) -> DSC1001DI2-012.0000T
Changed lines of the file:
@@
 F 2 "Package_BGA:BGA-256_14.0x14.0mm_Layout16x16_P0.8mm_Ball0.45mm_Pad0.32mm_NSMD" H 11250 2200 50  0001 C CNN
 F 3 "" H 11250 2200 50  0001 C CNN
+F 4 "Lattice" H 11250 2200 50  0001 C CNN "Manufacturer"
+F 5 "iCE40HX8K-CT256" H 11250 2200 50  0001 C CNN "Part number"
 	2    11250 2200
 	1    0    0    -1
@@
 Wire Wire Line
 	6300 7350 6300 7500
-$Comp
-L Interface_USB:FT2232H U?
-U 1 1 5D1FBC59
-P 6900 5150
-F 0 "U?" H 6000 7400 50  0000 C CNN
-F 1 "FT2232H" H 6000 7300 50  0000 C CNN
-F 2 "" H 6900 5150 50  0001 C CNN
-F 3 "http://www.ftdichip.com/Products/ICs/FT2232H.html" H 6900 5150 50  0001 C CNN
-	1    6900 5150
-	1    0    0    -1
-$EndComp
 Wire Wire Line
 	7400 2650 7400 2750
@@
 F 0 "U?" H 1850 5750 50  0000 C CNN
 F 1 "93LC56C-I_SN" H 1850 5250 50  0000 C CNN
-F 2 "" H 1850 5750 50  0001 C CNN
+F 2 "Package_SO:SOIC-8_3.9x4.9mm_P1.27mm" H 1850 5750 50  0001 C CNN
 F 3 "http://ww1.microchip.com/downloads/en/DeviceDoc/21794G.pdf" H 1850 5750 50  0001 C CNN
+F 4 "Microchip " H 1850 5750 50  0001 C CNN "Manufacturer"
+F 5 "93LC56C-I/SN " H 1850 5750 50  0001 C CNN "Part number"
 	1    1850 5750
 	-1   0    0    -1
@@
 F 0 "X?" H 3150 6850 50  0000 C CNN
 F 1 "DSC1001DI2-012.0000" H 3150 6450 50  0000 C CNN
-F 2 "" H 3250 6900 50  0001 C CNN
+F 2 "Crystal:Crystal_SMD_2520-4Pin_2.5x2.0mm" H 3250 6900 50  0001 C CNN
 F 3 "https://ww1.microchip.com/downloads/en/DeviceDoc/20005529B.pdf" H 3250 6900 50  0001 C CNN
+F 4 "Microchip" H 3150 6850 50  0001 C CNN "Manufacturer"
+F 5 "DSC1001DI2-012.0000T" H 3150 6850 50  0001 C CNN "Part number"
 	1    3150 6850
 	1    0    0    -1
@@
 F 0 "U?" H 13350 3350 50  0000 C CNN
 F 1 "AT25SF041-SSHD" H 13350 2750 50  0000 C CNN
-F 2 "" H 13350 3350 50  0001 C CNN
+F 2 "Package_SO:SOIC-8_3.9x4.9mm_P1.27mm" H 13350 3350 50  0001 C CNN
 F 3 "https://www.adestotech.com/wp-content/uploads/DS-AT25SF041_044.pdf" H 13350 3350 50  0001 C CNN
+F 4 "Adesto Technologies " H 13350 3350 50  0001 C CNN "Manufacturer"
+F 5 "AT25SF041-SSHD-B " H 13350 3350 50  0001 C CNN "Part number"
 	1    13350 3350
 	1    0    0    -1
@@
 Wire Wire Line
 	1075 1500 1425 1500
+$Comp
+L icenes-library:FT2232H U?
+U 1 1 5D4C9481
+P 6900 5150
+F 0 "U?" H 6900 7531 50  0000 C CNN
+F 1 "FT2232H" H 6900 7440 50  0000 C CNN
+F 2 "Package_QFP:LQFP-64_10x10mm_P0.5mm" H 6900 5150 50  0001 C CNN
+F 3 "http://www.ftdichip.com/Products/ICs/FT2232H.html" H 6900 5150 50  0001 C CNN
+F 4 "FTDI" H 6900 5150 50  0001 C CNN "Manufacturer"
+F 5 "FT2232HL" H 6900 5150 50  0001 C CNN "Part number"
+	1    6900 5150
+	1    0    0    -1
+$EndComp
 $EndSCHEMATC

Commit message: Footprints.
Parts:
- removed TP? (x2): TestPoint, symbol Connector:TestPoint
- added TP? (x2): TestPoint, TestPoint:TestPoint_Pad_D1.0mm, symbol icenes-library:TestPoint
Changed lines of the file:
@@
 	1775 1500 1825 1500
-$Comp
-L Connector:TestPoint TP?
-U 1 1 5D3FF502
-P 1825 1425
-AR Path="/5D3FF502" Ref="TP?"  Part="1"
-AR Path="/5D1BAC88/5D3FF502" Ref="TP?"  Part="1"
-F 0 "TP?" H 1900 1625 50  0000 R CNN
-F 1 "TestPoint" H 1767 1542 50  0001 R CNN
-F 2 "" H 2025 1425 50  0001 C CNN
-F 3 "~" H 2025 1425 50  0001 C CNN
-	1    1825 1425
-	1    0    0    -1
-$EndComp
 $Comp
 L icenes-library:R0 R?
@@
 F 6 "RC0805FR-070RL" H 1625 1500 50  0001 C CNN "Part number"
 	1    1625 1500
-	1    0    0    -1
-$EndComp
-$Comp
-L Connector:TestPoint TP?
-U 1 1 5D3FF511
-P 1425 1425
-AR Path="/5D3FF511" Ref="TP?"  Part="1"
-AR Path="/5D1BAC88/5D3FF511" Ref="TP?"  Part="1"
-F 0 "TP?" H 1500 1625 50  0000 R CNN
-F 1 "TestPoint" H 1367 1542 50  0001 R CNN
-F 2 "" H 1625 1425 50  0001 C CNN
-F 3 "~" H 1625 1425 50  0001 C CNN
-	1    1425 1425
 	1    0    0    -1
 $EndComp
@@
 U 1 1 5D4C9481
 P 6900 5150
-F 0 "U?" H 6900 7531 50  0000 C CNN
-F 1 "FT2232H" H 6900 7440 50  0000 C CNN
+F 0 "U?" H 5950 7325 50  0000 C CNN
+F 1 "FT2232H" H 6075 7250 50  0000 C CNN
 F 2 "Package_QFP:LQFP-64_10x10mm_P0.5mm" H 6900 5150 50  0001 C CNN
 F 3 "http://www.ftdichip.com/Products/ICs/FT2232H.html" H 6900 5150 50  0001 C CNN
@@
 	1    0    0    -1
 $EndComp
+$Comp
+L icenes-library:TestPoint TP?
+U 1 1 5D76AD94
+P 1425 1425
+AR Path="/5D76AD94" Ref="TP?"  Part="1"
+AR Path="/5D1BAC88/5D76AD94" Ref="TP?"  Part="1"
+F 0 "TP?" H 1375 1625 50  0000 L CNN
+F 1 "TestPoint" H 1425 1625 50  0001 C CNN
+F 2 "TestPoint:TestPoint_Pad_D1.0mm" H 1625 1425 50  0001 C CNN
+F 3 "~" H 1625 1425 50  0001 C CNN
+	1    1425 1425
+	1    0    0    -1
+$EndComp
+$Comp
+L icenes-library:TestPoint TP?
+U 1 1 5D773D53
+P 1825 1425
+AR Path="/5D773D53" Ref="TP?"  Part="1"
+AR Path="/5D1BAC88/5D773D53" Ref="TP?"  Part="1"
+F 0 "TP?" H 1775 1625 50  0000 L CNN
+F 1 "TestPoint" H 1825 1625 50  0001 C CNN
+F 2 "TestPoint:TestPoint_Pad_D1.0mm" H 2025 1425 50  0001 C CNN
+F 3 "~" H 2025 1425 50  0001 C CNN
+	1    1825 1425
+	1    0    0    -1
+$EndComp

Commit message: Completed USB interface. Clock sources for PAL and NTSC frequencies. Added a 133MHz clock (max input to PLL). Some more stuff.
Parts:
- removed C? (x3): C0.1uF, Capacitor_SMD:C_0603_1608Metric_Pad1.05x0.95mm_HandSolder, symbol icenes-library:C0.1uF
- added FB? (x2): FB600_500mA_0603, Inductor_SMD:L_0603_1608Metric_Pad1.05x0.95mm_HandSolder, symbol icenes-library:FB600_500mA_0603
- added R?: R10K, Resistor_SMD:R_0603_1608Metric_Pad1.05x0.95mm_HandSolder, symbol icenes-library:R10K
- added R?: R4.7K, Resistor_SMD:R_0603_1608Metric_Pad1.05x0.95mm_HandSolder, symbol icenes-library:R4.7K
Connections:
- net +3V3_FTDI: now also FB?.1, FB?.2, R?.1; no longer C?.1, C?.1, C?.1, C?.1, U?.4 (VPHY), U?.9 (VPLL)
- net GND: now also R?.2
- net ICE_CLK_12MHZ: now reaches U?.2 (OSCI), X?.3 (OUT)
- net at U?.59 (BCBUS7): now also R?.1, R?.2
- new net: C?.1, C?.1, FB?.1, U?.4 (VPHY)
- new net: C?.1, C?.1, FB?.2, U?.9 (VPLL)
- no-connect marks 23 -> 22
Other:
- moved on the sheet: C?, R?, TP?

Commit message: Minor fixes.
Parts:
- gave numbers to parts that had none: 34

Commit message: Fixed all ECR warnings.
Parts:
- removed C34, C36: C0.1uF, Capacitor_SMD:C_0603_1608Metric_Pad1.05x0.95mm_HandSolder, symbol icenes-library:C0.1uF
- removed R12: R0, Resistor_SMD:R_0805_2012Metric_Pad1.15x1.40mm_HandSolder, symbol icenes-library:R0
- removed TP15, TP16: TestPoint, TestPoint:TestPoint_Pad_D1.0mm, symbol icenes-library:TestPoint
- renumbered C35 to C36
