File: hw/icenes.kicad_pcb (KiCad board)
At the start: 6 copper layers, 100 x 100 mm, 201 parts, among them J1 USB_B_Micro, J2 Barrel_Jack_Switch, J3 Conn_02x11_Odd_Even, J4 Conn_02x31_Odd_Even, J5 Conn_02x31_Odd_Even, J6 NES-Connector-72pin, U1 TPS62050, U10 74ALVC164245, U11 74ALVC164245, U12 74ALVC164245, U13 74ALVC164245, U2 TPS62050, U3 TPS62056, U4 iCE40HX8K-CT256, U5 93LC56C-I_SN, U6 FT2232H, U7 AT25SF041-SSHD, U8 SN74LVC1404, U9 SN74LVC1404, X1 DSC1001DI2-012.0000, Y1 21.47727MHz, Y2 26.601712MHz

Commit message: Layout.
Parts:
- moved C73 21.7 mm to (101.5, 89.0), turned to 180 degrees
- moved C53 21.3 mm to (101.0, 110.0)
- moved C76 19.5 mm to (101.5, 90.6), turned to 180 degrees
- moved C50 17.7 mm to (102.5, 110.0)
- moved C72 10.1 mm to (120.2, 95.5)
- moved C44 9.82 mm to (121.5, 93.1)
- moved C86 3.95 mm to (118.5, 91.0)
- moved C46 1.88 mm to (115.8, 94.5)
Connections:
- J3 pad 10: Net-(J3-Pad10) -> GPIO_G14
- J3 pad 11: Net-(J3-Pad11) -> /ICENES io2/GPIO_K11
- J3 pad 12: Net-(J3-Pad12) -> GPIO_J10
- J3 pad 13: Net-(J3-Pad13) -> /ICENES io2/GPIO_P7
- J3 pad 14: Net-(J3-Pad14) -> GPIO_H11
- J3 pad 15: Net-(J3-Pad15) -> /ICENES io2/GPIO_R2
- J3 pad 16: Net-(J3-Pad16) -> /ICENES io2/GPIO_T1
- J3 pad 17: Net-(J3-Pad17) -> /ICENES io2/GPIO_R3
- J3 pad 18: Net-(J3-Pad18) -> /ICENES io2/GPIO_T2
- J3 pad 19: Net-(J3-Pad19) -> /ICENES io2/GPIO_R4
- J3 pad 20: Net-(J3-Pad20) -> /ICENES io2/GPIO_T3
- J3 pad 21: Net-(J3-Pad21) -> /ICENES io2/GPIO_T5
- J3 pad 22: Net-(J3-Pad22) -> /ICENES io2/GPIO_R5
- J3 pad 7: Net-(J3-Pad7) -> /ICENES io2/GPIO_P2
- J3 pad 8: Net-(J3-Pad8) -> /ICENES io2/GPIO_M5
- J3 pad 9: Net-(J3-Pad9) -> /ICENES io2/GPIO_R1
- J4 pad 10: Net-(J4-Pad10) -> /ICENES io2/GPIO_P5
- J4 pad 11: Net-(J4-Pad11) -> /ICENES io2/GPIO_N5
- J4 pad 12: Net-(J4-Pad12) -> /ICENES io2/GPIO_P6
- J4 pad 13: Net-(J4-Pad13) -> /ICENES io2/GPIO_N6
- J4 pad 14: Net-(J4-Pad14) -> /ICENES io2/GPIO_M7
- J4 pad 15: Net-(J4-Pad15) -> /ICENES io2/GPIO_N7
- J4 pad 16: Net-(J4-Pad16) -> /ICENES io2/GPIO_M8
- J4 pad 17: Net-(J4-Pad17) -> /ICENES io2/GPIO_T7
- J4 pad 18: Net-(J4-Pad18) -> /ICENES io2/GPIO_P8
- J4 pad 19: Net-(J4-Pad19) -> /ICENES io2/GPIO_P9
- J4 pad 7: Net-(J4-Pad7) -> /ICENES io2/GPIO_R6
- J4 pad 8: Net-(J4-Pad8) -> /ICENES io2/GPIO_T6
- J4 pad 9: Net-(J4-Pad9) -> /ICENES io2/GPIO_P4
- J5 pad 10: Net-(J5-Pad10) -> /ICENES io2/GPIO_N3
- J5 pad 11: Net-(J5-Pad11) -> /ICENES io2/GPIO_M6
- J5 pad 12: Net-(J5-Pad12) -> /ICENES io2/GPIO_M3
- J5 pad 13: Net-(J5-Pad13) -> /ICENES io2/GPIO_L7
- J5 pad 14: Net-(J5-Pad14) -> /ICENES io2/GPIO_N2
- J5 pad 15: Net-(J5-Pad15) -> /ICENES io2/GPIO_K5
- J5 pad 16: Net-(J5-Pad16) -> /ICENES io2/GPIO_M2
- J5 pad 17: Net-(J5-Pad17) -> /ICENES io2/GPIO_L6
- J5 pad 18: Net-(J5-Pad18) -> /ICENES io2/GPIO_L3
- J5 pad 19: Net-(J5-Pad19) -> /ICENES io2/GPIO_K4
- J5 pad 20: Net-(J5-Pad20) -> /ICENES io2/GPIO_M1
- J5 pad 21: Net-(J5-Pad21) -> /ICENES io2/GPIO_L4
- J5 pad 22: Net-(J5-Pad22) -> /ICENES io2/GPIO_L1
- J5 pad 23: Net-(J5-Pad23) -> /ICENES io2/GPIO_K1
- J5 pad 24: Net-(J5-Pad24) -> /ICENES io2/GPIO_K3
- J5 pad 25: Net-(J5-Pad25) -> /ICENES io2/GPIO_J2
- J5 pad 26: Net-(J5-Pad26) -> /ICENES io2/GPIO_J1
- J5 pad 27: Net-(J5-Pad27) -> /ICENES io2/GPIO_J5
- J5 pad 28: Net-(J5-Pad28) -> /ICENES io2/GPIO_H1
- J5 pad 29: Net-(J5-Pad29) -> /ICENES io2/GPIO_J4
- J5 pad 30: Net-(J5-Pad30) -> /ICENES io2/GPIO_H2
- J5 pad 33: Net-(J5-Pad33) -> /ICENES io2/GPIO_N4
- J5 pad 35: Net-(J5-Pad35) -> /ICENES io2/GPIO_H4
- J5 pad 36: Net-(J5-Pad36) -> /ICENES io2/GPIO_G2
- J5 pad 37: Net-(J5-Pad37) -> /ICENES io2/GPIO_H6
- J5 pad 38: Net-(J5-Pad38) -> /ICENES io2/GPIO_F1
- J5 pad 39: Net-(J5-Pad39) -> /ICENES io2/GPIO_H3
- J5 pad 40: Net-(J5-Pad40) -> /ICENES io2/GPIO_F2
- J5 pad 41: Net-(J5-Pad41) -> /ICENES io2/GPIO_G3
- J5 pad 42: Net-(J5-Pad42) -> /ICENES io2/GPIO_F3
- J5 pad 43: Net-(J5-Pad43) -> /ICENES io2/GPIO_H5
- J5 pad 44: Net-(J5-Pad44) -> /ICENES io2/GPIO_E2
- J5 pad 45: Net-(J5-Pad45) -> /ICENES io2/GPIO_G4
- J5 pad 46: Net-(J5-Pad46) -> /ICENES io2/GPIO_E3
- J5 pad 47: Net-(J5-Pad47) -> /ICENES io2/GPIO_G5
- J5 pad 48: Net-(J5-Pad48) -> /ICENES io2/GPIO_D1
- J5 pad 49: Net-(J5-Pad49) -> /ICENES io2/GPIO_F4
- J5 pad 50: Net-(J5-Pad50) -> /ICENES io2/GPIO_D2
- J5 pad 51: Net-(J5-Pad51) -> /ICENES io2/GPIO_C1
- J5 pad 52: Net-(J5-Pad52) -> /ICENES io2/GPIO_C2
- J5 pad 53: Net-(J5-Pad53) -> /ICENES io2/GPIO_F5
- J5 pad 54: Net-(J5-Pad54) -> /ICENES io2/GPIO_B1
- J5 pad 55: Net-(J5-Pad55) -> /ICENES io2/GPIO_E4
- J5 pad 56: Net-(J5-Pad56) -> /ICENES io2/GPIO_B2
- J5 pad 7: Net-(J5-Pad7) -> /ICENES io2/GPIO_P1
- J5 pad 8: Net-(J5-Pad8) -> /ICENES io2/GPIO_M4
- J5 pad 9: Net-(J5-Pad9) -> /ICENES io2/GPIO_L5
- U4 pad G14: /ICENES io1/GPIO_G14 -> GPIO_G14
- U4 pad H11: /ICENES io1/GPIO_H11 -> GPIO_H11
- U4 pad J10: /ICENES io1/GPIO_C10 -> GPIO_J10
Routing:
- net /ICENES io2/GPIO_N4: track 3.78 -> 95.2 mm
- net /ICENES io2/GPIO_T6: track 2.10 -> 74.5 mm, vias 0 -> 1
- net /ICENES io2/GPIO_R6: track 3.49 -> 72.5 mm, vias 0 -> 1
- net /ICENES io2/GPIO_P5: track 2.87 -> 70.8 mm
- net /ICENES io2/GPIO_P4: track 2.82 -> 68.3 mm
- net /ICENES io2/GPIO_P8: track 3.03 -> 68.1 mm
- net /ICENES io2/GPIO_N5: track 3.78 -> 67.8 mm
- net /ICENES io2/GPIO_P6: track 2.82 -> 66.7 mm
- net /ICENES io2/GPIO_P1: track 1.10 -> 64.9 mm
- net GPIO_J10: track 0.00 -> 63.3 mm, vias 0 -> 2
- net /ICENES io2/GPIO_T7: track 2.10 -> 65.2 mm, vias 0 -> 1
- net /ICENES io2/GPIO_P9: track 3.03 -> 63.8 mm
- net GPIO_H11: track 0.00 -> 60.7 mm, vias 0 -> 2
- net /ICENES io2/GPIO_M7: track 4.58 -> 64.8 mm
- net /ICENES io2/GPIO_N6: track 3.83 -> 63.2 mm
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
Commit message: Layout.
Parts:
- C32, C34: moved to B.Cu
- moved C20 110.6 mm to (63.5, 70.2)
- moved C16 102.3 mm to (77.0, 69.6), turned to 180 degrees
- moved C34 64.0 mm to (93.9, 106.6), turned to 180 degrees
- moved C32 62.7 mm to (93.9, 108.3), turned to 180 degrees
- moved C25 53.8 mm to (110.5, 84.2), turned to 180 degrees
- moved C22 51.1 mm to (110.5, 85.9), turned to 180 degrees
- moved C30 47.4 mm to (112.5, 99.6)
- moved C28 46.6 mm to (112.5, 97.9)
- moved C18 46.3 mm to (113.9, 85.9)
- moved C14 45.9 mm to (113.9, 84.2)
Routing:
- net GND: track 240.4 -> 249.0 mm, vias 81 -> 87
- net +1V2: track 269.1 -> 276.7 mm, vias 12 -> 15
- net /ICENES io2/GPIO_G2: track 43.9 -> 46.4 mm
- net +3V3_FTDI: track 50.7 -> 52.7 mm, vias 10 -> 11
- net /ICENES io2/GPIO_F1: track 41.9 -> 43.2 mm

Commit message: Layout.
Parts:
- moved C46 43.9 mm to (159.1, 102.2)
- moved C58 43.9 mm to (161.8, 102.0)
- moved C72 43.9 mm to (163.4, 103.3)
- moved C44 43.9 mm to (164.7, 100.9)
- moved C86 43.9 mm to (161.7, 98.8)
- moved D2 5.46 mm to (91.1, 107.6)
- moved C50 0.54 mm to (102.8, 109.5)
- moved C53 0.50 mm to (101.0, 109.5)
Connections:
- J3 pad 10: GPIO_G14 -> /ICENES io2/GPIO_P2
- J3 pad 11: /ICENES io2/GPIO_K11 -> /ICENES io2/GPIO_R3
- J3 pad 12: GPIO_J10 -> /ICENES io2/GPIO_T2
- J3 pad 13: /ICENES io2/GPIO_P7 -> /ICENES io2/GPIO_T3
- J3 pad 14: GPIO_H11 -> /ICENES io2/GPIO_P4
- J3 pad 15: /ICENES io2/GPIO_R2 -> /ICENES io2/GPIO_R4
- J3 pad 16: /ICENES io2/GPIO_T1 -> /ICENES io2/GPIO_N5
- J3 pad 17: /ICENES io2/GPIO_R3 -> /ICENES io2/GPIO_R5
- J3 pad 18: /ICENES io2/GPIO_T2 -> /ICENES io2/GPIO_P5
- J3 pad 19: /ICENES io2/GPIO_R4 -> /ICENES io2/GPIO_P6
- J3 pad 20: /ICENES io2/GPIO_T3 -> /ICENES io2/GPIO_T5
- J3 pad 21: /ICENES io2/GPIO_T5 -> /ICENES io2/GPIO_T6
- J3 pad 22: /ICENES io2/GPIO_R5 -> /ICENES io2/GPIO_R6
- J3 pad 7: /ICENES io2/GPIO_P2 -> /ICENES io2/GPIO_T1
- J3 pad 8: /ICENES io2/GPIO_M5 -> /ICENES io2/GPIO_R1
- J3 pad 9: /ICENES io2/GPIO_R1 -> /ICENES io2/GPIO_R2
- J4 pad 10: /ICENES io2/GPIO_P5 -> /ICENES io2/GPIO_M7
- J4 pad 11: /ICENES io2/GPIO_N5 -> /ICENES io2/GPIO_N7
- J4 pad 12: /ICENES io2/GPIO_P6 -> /ICENES io2/GPIO_M8
- J4 pad 13: /ICENES io2/GPIO_N6 -> /ICENES io2/GPIO_T11
- J4 pad 14: /ICENES io2/GPIO_M7 -> /ICENES io2/GPIO_P10
- J4 pad 15: /ICENES io2/GPIO_N7 -> /ICENES io2/GPIO_R10
- J4 pad 16: /ICENES io2/GPIO_M8 -> /ICENES io2/GPIO_T10
- J4 pad 17: /ICENES io2/GPIO_T7 -> /ICENES io2/GPIO_T13
- J4 pad 18: /ICENES io2/GPIO_P8 -> /ICENES io2/GPIO_P13
- J4 pad 19: /ICENES io2/GPIO_P9 -> /ICENES io2/GPIO_T14
- J4 pad 20: /ICENES io2/GPIO_M9 -> GPIO_R14
- J4 pad 21: /ICENES io2/GPIO_L9 -> /ICENES io2/GPIO_T15
- J4 pad 22: /ICENES io2/GPIO_L10 -> GPIO_R15
- J4 pad 23: /ICENES io2/GPIO_M11 -> /ICENES io2/GPIO_T16
- J4 pad 24: /ICENES io2/GPIO_M12 -> GPIO_P14
- J4 pad 25: /ICENES io2/GPIO_T11 -> /ICENES io2/GPIO_R16
- J4 pad 26: /ICENES io2/GPIO_L11 -> GPIO_P15
- J4 pad 27: /ICENES io2/GPIO_T14 -> GPIO_M13
- J4 pad 28: /ICENES io2/GPIO_T13 -> GPIO_P16
- J4 pad 29: /ICENES io2/GPIO_T16 -> GPIO_N16
- J4 pad 30: /ICENES io2/GPIO_T15 -> GPIO_M14
- J4 pad 33: GPIO_R14 -> GPIO_M15
- J4 pad 35: GPIO_P14 -> GPIO_L14
- J4 pad 36: /ICENES io2/GPIO_P13 -> GPIO_M16
- J4 pad 37: GPIO_M13 -> GPIO_K14
- J4 pad 38: /ICENES io2/GPIO_N12 -> GPIO_L16
- J4 pad 39: GPIO_L14 -> GPIO_K16
- J4 pad 40: GPIO_M14 -> GPIO_K15
- J4 pad 41: GPIO_K14 -> GPIO_J10
- J4 pad 42: GPIO_K13 -> GPIO_J14
- J4 pad 43: GPIO_J14 -> /ICENES io2/GPIO_L9
- J4 pad 44: GPIO_J13 -> /ICENES io2/GPIO_L10
- J4 pad 45: GPIO_R15 -> /ICENES io2/GPIO_N10
- J4 pad 46: GPIO_H12 -> /ICENES io2/GPIO_M9
- J4 pad 47: GPIO_P15 -> GPIO_J16
- J4 pad 48: /ICENES io2/GPIO_R16 -> GPIO_J15
- J4 pad 49: GPIO_N16 -> /ICENES io2/GPIO_M11
- J4 pad 50: GPIO_P16 -> /ICENES io2/GPIO_N12
- J4 pad 51: GPIO_L12 -> /ICENES io2/GPIO_L11
- J4 pad 52: GPIO_M15 -> /ICENES io2/GPIO_M12
- J4 pad 53: GPIO_K12 -> GPIO_L12
- J4 pad 55: GPIO_J11 -> GPIO_K12
- J4 pad 56: GPIO_J12 -> GPIO_K13
- J4 pad 7: /ICENES io2/GPIO_R6 -> /ICENES io2/GPIO_N4
- J4 pad 8: /ICENES io2/GPIO_T6 -> /ICENES io2/GPIO_M5
- J4 pad 9: /ICENES io2/GPIO_P4 -> /ICENES io2/GPIO_N6
- J5 pad 33: /ICENES io2/GPIO_N4 -> /ICENES io2/GPIO_K9
- TP15 pad 1: /ICENES io1/ICE_CLK_26.601712MHz -> ICE_CLK_26.601712MHz
- U4 pad A1: ICE_CPU_RW -> ICE_CPU_A3
- U4 pad A10: ICE_PPU_A9 -> ICE_PPU_A4
- U4 pad A11: ICE_PPU_A7 -> ICE_PPU_A1
- U4 pad A15: ICE_PPU_D7 -> ICE_PPU_D2
- U4 pad A16: ICE_PPU_D6 -> ICE_PPU_D0
- U4 pad A2: ICE_CPU_A13 -> ICE_CPU_A2
- U4 pad A5: ICE_CPU_A9 -> ~ICE_PPU_A13
- U4 pad A6: ICE_CPU_A7 -> ICE_PPU_A12
- U4 pad A7: ICE_CPU_A3 -> ICE_PPU_A9
- U4 pad A9: ICE_PPU_A13 -> ICE_PPU_A6
- U4 pad B10: ICE_PPU_A8 -> ICE_PPU_A3
- U4 pad B11: ICE_PPU_A1 -> ICE_PPU_A0
- U4 pad B12: ICE_PPU_A0 -> ICE_PPU_D7
- U4 pad B13: PPU_DATA_DIR -> ICE_PPU_D5
- U4 pad B14: ~PPU_DATA_OE -> /ICENES io1/LED2
- U4 pad B15: ICE_PPU_D0 -> ICE_PPU_D1
- U4 pad B3: ICE_CPU_A8 -> ICE_CPU_A0
- U4 pad B4: ICE_CPU_A12 -> CPU_ADDR_DIR
- U4 pad B5: ICE_CPU_A10 -> ~ICE_PPU_WR
- U4 pad B6: ICE_CPU_A4 -> /ICENES io1/LED6
- U4 pad B7: ICE_CPU_A1 -> ICE_PPU_A10
- U4 pad B8: ICE_CPU_A0 -> ICE_PPU_A7
- U4 pad B9: ICE_PPU_A11 -> ICE_PPU_A5
- U4 pad C10: ICE_PPU_A6 -> ICE_PPU_A2
- U4 pad C11: ICE_PPU_A5 -> ~PPU_ADDR_OE
- U4 pad C12: ~PPU_ADDR_OE -> ICE_PPU_D6
- U4 pad C13: PPU_ADDR_DIR -> ICE_PPU_D4
- U4 pad C14: ICE_PPU_D1 -> ICE_PPU_D3
- U4 pad C3: ICE_CPU_A11 -> ICE_CPU_A1
- U4 pad C4: ICE_CPU_A6 -> ~CPU_ADDR_OE
- U4 pad C5: ICE_CPU_A5 -> /ICENES io1/LED7
- U4 pad C6: ~CPU_ADDR_OE -> ICE_PPU_A13
- U4 pad C7: ~ICE_PPU_WR -> ICE_PPU_A11
- U4 pad C8: ~ICE_PPU_A13 -> ICE_PPU_A8
- U4 pad C9: ICE_PPU_A10 -> /ICENES io1/LED5
- U4 pad D10: /ICENES io1/LED4 -> ICE_CPU_A4
- U4 pad D11: /ICENES io1/LED3 -> PPU_ADDR_DIR
- U4 pad D13: /ICENES io1/LED1 -> ~PPU_DATA_OE
- U4 pad D14: ICE_CPU_D4 -> ICE_CPU_D5
- U4 pad D15: ICE_CPU_D5 -> ICE_CPU_D4
- U4 pad D16: ICE_CPU_D2 -> /ICENES io1/LED1
- U4 pad D3: ICE_CPU_A14 -> Net-(U4-PadD3)
- U4 pad D4: /ICENES io1/LED7 -> ICE_CPU_RW
- U4 pad D5: /ICENES io1/LED6 -> ICE_CPU_A13
- U4 pad D6: ICE_CPU_A2 -> ICE_CPU_A11
- U4 pad D7: CPU_ADDR_DIR -> ICE_CPU_A10
- U4 pad D8: ICE_PPU_A3 -> ICE_CPU_A9
- U4 pad D9: ICE_PPU_A12 -> ICE_CPU_A6
- U4 pad E10: ICE_PPU_D4 -> ICE_CPU_A5
- U4 pad E11: /ICENES io1/LED2 -> /ICENES io1/LED3
- U4 pad E13: ICE_CICtoMB -> ICE_CIRAM_A10
- U4 pad E16: ICE_CPU_D1 -> ICE_CPU_D2
- U4 pad E5: /ICENES io1/LED5 -> ICE_CPU_A14
- U4 pad E6: ICE_PPU_A4 -> ICE_CPU_A12
- U4 pad E9: ICE_PPU_A2 -> ICE_CPU_A7
- U4 pad F11: /ICENES io1/LED0 -> PPU_DATA_DIR
- U4 pad F12: ICE_M2 -> ICE_CICtoMB
- U4 pad F13: ~ICE_CIC_RST -> ~ICE_IRQ
- U4 pad F14: CPU_DATA_DIR -> ICE_CPU_D1
- U4 pad F15: ICE_CIRAM_A10 -> ICE_CPU_D0
- U4 pad F16: ICE_CPU_D0 -> ~CPU_DATA_OE
- U4 pad F7: /ICENES io1/ICE_CLK_26.601712MHz -> Net-(U4-PadF7)
- U4 pad F9: ICE_PPU_D5 -> ICE_CPU_A8
- U4 pad G1: Net-(U4-PadG1) -> ICE_CLK_26.601712MHz
- U4 pad G10: ICE_PPU_D3 -> /ICENES io1/LED4
- U4 pad G11: ICE_PPU_D2 -> ~ICE_CIRAM_CE
- U4 pad G12: ICE_SYSTEM_CLK -> ICE_CICtoPak
- U4 pad G13: ICE_CICtoPak -> ~ICE_CIC_RST
- U4 pad G14: GPIO_G14 -> CPU_DATA_DIR
- U4 pad G15: ~ICE_CIRAM_CE -> /ICENES io1/LED0
- U4 pad G16: ~CPU_DATA_OE -> MISC_DIR2
- U4 pad H11: GPIO_H11 -> ~ICE_PPU_RD
- U4 pad H12: GPIO_H12 -> ~ICE_ROMSEL
- U4 pad H14: ~ICE_IRQ -> ~MISC_OE2
- U4 pad J11: GPIO_J11 -> ICE_SYSTEM_CLK
- U4 pad J12: GPIO_J12 -> ~MISC_OE1
- U4 pad J13: GPIO_J13 -> MISC_DIR1
- U4 pad J15: ~MISC_OE2 -> GPIO_J15
- U4 pad J16: MISC_DIR2 -> GPIO_J16
- U4 pad J3: ICE_CLK_12MHZ -> Net-(U4-PadJ3)
- U4 pad K11: /ICENES io2/GPIO_K11 -> ICE_M2
- U4 pad K15: ~ICE_PPU_RD -> GPIO_K15
- U4 pad K16: ~ICE_ROMSEL -> GPIO_K16
- U4 pad K9: Net-(U4-PadK9) -> /ICENES io2/GPIO_K9
- U4 pad L16: ~MISC_OE1 -> GPIO_L16
- U4 pad M16: MISC_DIR1 -> GPIO_M16
- U4 pad N10: DTRn -> /ICENES io2/GPIO_N10
- U4 pad N9: DCDn -> RS232_RX_TTL
- U4 pad P10: DSRn -> /ICENES io2/GPIO_P10
- U4 pad P7: /ICENES io2/GPIO_P7 -> DCDn
- U4 pad P8: /ICENES io2/GPIO_P8 -> DTRn
- U4 pad P9: /ICENES io2/GPIO_P9 -> RS232_TX_TTL
- U4 pad R10: RS232_TX_TTL -> /ICENES io2/GPIO_R10
- U4 pad R9: Net-(U4-PadR9) -> ICE_CLK_12MHZ
- U4 pad T10: RS232_RX_TTL -> /ICENES io2/GPIO_T10
- U4 pad T7: /ICENES io2/GPIO_T7 -> DSRn
- U9 pad 7: /ICENES io1/ICE_CLK_26.601712MHz -> ICE_CLK_26.601712MHz
Routing:
- net /ICENES io2/GPIO_N10: track 0.00 -> 69.7 mm, vias 0 -> 1
- net /ICENES io2/GPIO_P8: track 68.1 -> 0.00 mm, vias 1 -> 0
- net /ICENES io2/GPIO_T7: track 65.2 -> 0.00 mm, vias 1 -> 0
- net /ICENES io2/GPIO_P9: track 63.8 -> 0.00 mm, vias 1 -> 0
- net /ICENES io2/GPIO_P10: track 0.00 -> 63.8 mm, vias 0 -> 1
- net /ICENES io2/GPIO_T10: track 0.00 -> 61.9 mm, vias 0 -> 1
- net GPIO_H11: track 60.7 -> 0.00 mm, vias 2 -> 0
- net /ICENES io2/GPIO_R10: track 0.00 -> 59.7 mm, vias 0 -> 1
- net /ICENES io2/GPIO_K11: track 56.8 -> 0.00 mm, vias 2 -> 0
- net GPIO_G14: track 56.5 -> 0.00 mm, vias 2 -> 0
- net GPIO_J12: track 54.5 -> 0.00 mm, vias 1 -> 0
- net GPIO_J11: track 52.8 -> 0.00 mm, vias 1 -> 0
- net /ICENES io2/GPIO_K9: track 0.00 -> 51.9 mm, vias 0 -> 1
- net GPIO_H12: track 49.1 -> 0.00 mm, vias 1 -> 0
- net GPIO_J15: track 0.00 -> 49.1 mm, vias 0 -> 1
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Other:
- net class Default: clearance 0.127 -> 0.0889
- rule trace_clearance: 0.127 -> 0.0889

Commit message: Layout.
Parts:
- moved R14 2.18 mm to (64.2, 74.0), turned to 270 degrees
Routing:
- net USB_D_P: track 23.3 -> 38.6 mm, vias 2 -> 0
- net USB_D_N: track 23.1 -> 38.1 mm, vias 2 -> 0
- net +1V2: track 291.9 -> 291.2 mm
- net Net-(R14-Pad2): track 6.80 -> 7.38 mm

Commit message: Layout.
Parts:
- C44, C46, C58, C72, C86: moved to F.Cu
- moved C86 7.20 mm to (161.7, 106.0)
- moved C44 3.00 mm to (164.7, 103.9)
- moved C72 1.80 mm to (163.4, 101.5), turned to 90 degrees
- moved C58 0.80 mm to (161.8, 102.8), turned to 270 degrees
- moved C46 0.30 mm to (159.1, 102.5), turned to 90 degrees
Connections:
- U10 pad 12: /ICENES NES Connector/NES_PPU_A7 -> /ICENES NES Connector/NES_PPU_A13
- U10 pad 13: /ICENES NES Connector/NES_PPU_A8 -> /ICENES NES Connector/NES_PPU_A12
- U10 pad 14: /ICENES NES Connector/NES_PPU_A9 -> /ICENES NES Connector/NES_PPU_A10
- U10 pad 16: /ICENES NES Connector/NES_PPU_A10 -> /ICENES NES Connector/NES_PPU_A11
- U10 pad 17: /ICENES NES Connector/NES_PPU_A11 -> /ICENES NES Connector/NES_PPU_A9
- U10 pad 19: /ICENES NES Connector/NES_PPU_A12 -> /ICENES NES Connector/NES_PPU_A8
- U10 pad 20: /ICENES NES Connector/NES_PPU_A13 -> /ICENES NES Connector/NES_PPU_A7
- U10 pad 29: ICE_PPU_A13 -> ICE_PPU_A7
- U10 pad 30: ICE_PPU_A12 -> ICE_PPU_A8
- U10 pad 32: ICE_PPU_A11 -> ICE_PPU_A9
- U10 pad 33: ICE_PPU_A10 -> ICE_PPU_A11
- U10 pad 35: ICE_PPU_A9 -> ICE_PPU_A10
- U10 pad 36: ICE_PPU_A8 -> ICE_PPU_A12
- U10 pad 37: ICE_PPU_A7 -> ICE_PPU_A13
- U4 pad A6: ICE_PPU_A12 -> ICE_PPU_A8
- U4 pad A7: ICE_PPU_A9 -> ICE_PPU_A10
- U4 pad B7: ICE_PPU_A10 -> ICE_PPU_A11
- U4 pad B8: ICE_PPU_A7 -> ICE_PPU_A13
- U4 pad C6: ICE_PPU_A13 -> ICE_PPU_A7
- U4 pad C7: ICE_PPU_A11 -> ICE_PPU_A9
- U4 pad C8: ICE_PPU_A8 -> ICE_PPU_A12
Routing:
- net /ICENES NES Connector/NES_CIRAM_A10: track 26.0 -> 57.4 mm, vias 1 -> 0
- net /ICENES NES Connector/NES_CPU_RW: track 29.8 -> 56.5 mm, vias 1 -> 0
- net /ICENES NES Connector/~NES_CIRAM_CE: track 30.2 -> 55.0 mm, vias 1 -> 0
- net /ICENES NES Connector/NES_PPU_A7: track 51.6 -> 32.3 mm, vias 1 -> 0
- net /ICENES NES Connector/NES_PPU_A8: track 52.0 -> 34.4 mm, vias 1 -> 0
- net /ICENES NES Connector/NES_PPU_A10: track 55.3 -> 39.4 mm
- net /ICENES NES Connector/NES_PPU_A9: track 51.5 -> 36.3 mm
- net CPU_ADDR_DIR: track 39.8 -> 53.0 mm
- net PPU_ADDR_DIR: track 30.3 -> 43.1 mm
- net /ICENES NES Connector/NES_M2: track 115.3 -> 127.8 mm
- net /ICENES NES Connector/NES_CPU_A12: track 33.9 -> 21.6 mm
- net /ICENES NES Connector/NES_PPU_A12: track 53.6 -> 41.5 mm
- net /ICENES NES Connector/~NES_ROMSEL: track 86.4 -> 75.2 mm
- net /ICENES NES Connector/NES_PPU_A13: track 54.7 -> 43.7 mm
- net /ICENES NES Connector/NES_CPU_A13: track 34.6 -> 26.4 mm
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Other:
- rule trace_min: 0.0889 -> 0

Commit message: Layout.
Routing:
- net +5V: track 43.3 -> 34.7 mm
- net +3V3: track 113.9 -> 113.4 mm
- added copper zone on In2.Cu, net +1V2
- added copper zone on In2.Cu, net +3V3
- added copper zone on In2.Cu, net +3V3_FTDI
- added copper zone on In2.Cu, net +5V
- added copper zone on In2.Cu, net /Vin(+5V-+10V)
- added copper zone on In4.Cu, net GND
- removed copper zone on In4.Cu, net +1V2
- removed copper zone on In4.Cu, net +3V3
- removed copper zone on In4.Cu, net +3V3_FTDI
- removed copper zone on In4.Cu, net +5V
- removed copper zone on In4.Cu, net /Vin(+5V-+10V)

Commit message: Layout.
Parts:
- C23, C26: moved to B.Cu
- moved C13 107.2 mm to (79.2, 130.7), turned to 90 degrees
- moved C17 103.8 mm to (80.8, 130.7), turned to 90 degrees
- moved C59 86.3 mm to (81.4, 104.0), turned to 90 degrees
- moved C27 82.5 mm to (100.0, 130.7), turned to 90 degrees
- moved C72 80.2 mm to (83.2, 104.0)
- moved C63 78.1 mm to (88.5, 88.8), turned to 90 degrees
- moved C21 77.2 mm to (119.3, 130.7), turned to 90 degrees
- moved C35 77.0 mm to (85.8, 62.2)
- moved C44 77.0 mm to (88.0, 97.4)
- moved C82 75.6 mm to (83.2, 98.0), turned to 270 degrees
- moved C33 75.1 mm to (85.8, 63.8)
- moved C87 74.8 mm to (85.0, 98.0), turned to 270 degrees
- moved C46 74.1 mm to (85.0, 104.0)
- moved C24 73.7 mm to (121.0, 130.7), turned to 90 degrees
- moved C86 73.5 mm to (90.2, 88.8), turned to 90 degrees
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Routing:
- net GND: track 255.1 -> 281.8 mm, vias 158 -> 191
- net +3V3: track 113.4 -> 135.6 mm, vias 34 -> 59
- net +5V: track 34.7 -> 39.0 mm, vias 9 -> 14
- net /ICENES USB and flash/iCE_SCK: track 44.7 -> 47.1 mm
- net /ICENES NES Connector/NES_PPU_D0: track 24.5 -> 26.6 mm
- net /ICENES NES Connector/NES_PPU_D4: track 42.9 -> 45.0 mm
- net /ICENES NES Connector/NES_PPU_D3: track 34.6 -> 36.6 mm
- net /ICENES NES Connector/NES_PPU_D2: track 31.4 -> 33.4 mm
- net /ICENES NES Connector/NES_PPU_D1: track 27.7 -> 29.7 mm
- net +1V2: track 291.2 -> 291.3 mm, vias 16 -> 19
