File: hw/icenes.kicad_pcb (KiCad board)
At the start: 6 copper layers, 100 x 100 mm, 201 parts, among them J1 USB_B_Micro, J2 Barrel_Jack_Switch, J3 Conn_02x11_Odd_Even, J4 Conn_02x31_Odd_Even, J5 Conn_02x31_Odd_Even, J6 NES-Connector-72pin, U1 TPS62050, U10 74ALVC164245, U11 74ALVC164245, U12 74ALVC164245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

Commit message: Layout.  - Changed footprint of the nes connector from 2.54mm pitch and 5.08mm row pitch to 2.5mm pitch and 0.5mm row pitch.
Parts:
- J6: footprint icenes-library:DIP-72-NES-CONNECTOR-2 -> icenes-library:DIP-72-NES-CONNECTOR-3
- moved C106 1.30 mm to (55.3, 141.5)
Routing:
- net /ICENES NES Connector/NES_M2: track 127.8 -> 121.2 mm
- net /ICENES NES Connector/NES_SYSTEM_CLK: track 119.2 -> 113.2 mm
- net GND: track 281.8 -> 286.7 mm, vias 191 -> 196
- net /ICENES NES Connector/NES_CIRAM_A10: track 57.4 -> 55.4 mm
- net /ICENES NES Connector/NES_CPU_A2: track 11.4 -> 12.4 mm
- net /ICENES NES Connector/NES_CPU_A0: track 14.6 -> 15.5 mm
- net /ICENES NES Connector/NES_CPU_D5: track 47.2 -> 46.3 mm
- net /ICENES NES Connector/~NES_CIRAM_CE: track 55.0 -> 54.2 mm
- net /ICENES NES Connector/~NES_IRQ: track 52.0 -> 52.8 mm
- net /ICENES NES Connector/~NES_PPU_A13: track 31.3 -> 30.7 mm
- net /ICENES NES Connector/~NES_ROMSEL: track 75.2 -> 75.7 mm
- net /ICENES NES Connector/NES_CPU_D6: track 48.7 -> 48.2 mm
- net /ICENES NES Connector/NES_PPU_D6: track 34.6 -> 34.1 mm

Commit message: Layout. Cleaned up nes connector footprints. Adjusted LED (D1) series resistor. Adjusted the voltage divider to BCBUS7 on FT2232H. Set pull up resistor to CDONE to 10k.
Parts:
- J6: footprint icenes-library:DIP-72-NES-CONNECTOR-3 -> icenes-library:DIP-72-NES-CONNECTOR
- R1: value R2.2K -> R1.54k
- R16: value R4.7K -> R6.04k
- R36: value R_TBD -> R10K
Other:
- board text added: "1V2"
- board text added: "3V3"
- board text added: "5V"
- board text added: "B1"
- board text added: "B2"
- board text added: "C1"
- board text added: "C2"
- board text added: "D1"
- board text added: "D2"
- board text added: "E2"
- board text added: "E3"
- board text added: "E4"
- board text added: "F1"
- board text added: "F2"
- board text added: "F3"
- board text added: "F4"
- board text added: "F5"
- board text added: "G2"
- board text added: "G3"
- board text added: "G4"
- board text added: "G5"
- board text added: "GND"
- board text added: "H1"
- board text added: "H2"
- board text added: "H3"
- board text added: "H4"
- board text added: "H5"
- board text added: "H6"
- board text added: "J1"
- board text added: "J10"
- board text added: "J14"
- board text added: "J15"
- board text added: "J16"
- board text added: "J2"
- board text added: "J4"
- board text added: "J5"
- board text added: "K1"
- board text added: "K12"
- board text added: "K13"
- board text added: "K14"
- board text added: "K15"
- board text added: "K16"
- board text added: "K3"
- board text added: "K4"
- board text added: "K5"
- board text added: "K9"
- board text added: "L1"
- board text added: "L10"
- board text added: "L11"
- board text added: "L12"
- board text added: "L13"
- board text added: "L14"
- board text added: "L16"
- board text added: "L3"
- board text added: "L4"
- board text added: "L5"
- board text added: "L6"
- board text added: "L7"
- board text added: "L9"
- board text added: "M1"
- board text added: "M11"
- board text added: "M12"
- board text added: "M13"
- board text added: "M14"
- board text added: "M15"
- board text added: "M16"
- board text added: "M2"
- board text added: "M3"
- board text added: "M4"
- board text added: "M5"
- board text added: "M6"
- board text added: "M7"
- board text added: "M8"
- board text added: "M9"
- board text added: "N10"
- board text added: "N12"
- board text added: "N16"
- board text added: "N2"
- board text added: "N3"
- board text added: "N4"
- board text added: "N5"
- board text added: "N6"
- board text added: "N7"
- board text added: "P1"
- board text added: "P10"
- board text added: "P13"
- board text added: "P14"
- board text added: "P15"
- board text added: "P16"
- board text added: "P2"
- board text added: "P4"
- board text added: "P5"
- board text added: "P6"
- board text added: "R1"
- board text added: "R10"
- board text added: "R14"
- board text added: "R15"
- board text added: "R16"
- board text added: "R2"
- board text added: "R3"
- board text added: "R4"
- board text added: "R5"
- board text added: "R6"
- board text added: "T1"
- board text added: "T10"
- board text added: "T11"
- board text added: "T13"
- board text added: "T14"
- board text added: "T15"
- board text added: "T16"
- board text added: "T2"
- board text added: "T3"
- board text added: "T5"
- board text added: "T6"

Commit message: Added pwr led.
Parts:
- added D11: Green_LED, LED_SMD:LED_0805_2012Metric_Pad1.15x1.40mm_HandSolder, F.Cu at (119.9, 51.9)
- added R38: R698, Resistor_SMD:R_0603_1608Metric_Pad1.05x0.95mm_HandSolder, F.Cu at (119.9, 55.5)
- turned D1 to 270 degrees
Routing:
- net Net-(D11-Pad2): track 0.00 -> 1.72 mm
- net GND: track 286.7 -> 288.1 mm, vias 196 -> 197
- net Net-(D1-Pad2): track 3.32 -> 2.10 mm
- net +3V3: track 135.6 -> 136.5 mm, vias 59 -> 60
Other:
- board text added: "ICENES"
- board text added: "PWR"
- board text added: "Prototype 1"
- board text added: "USB"
