File: hw/icenes-io2.sch (KiCad schematic (older format))
At the start: 35 parts, among them J3 Conn_02x11_Odd_Even, J4 Conn_02x31_Odd_Even, J5 Conn_02x31_Odd_Even, U4 iCE40HX8K-CT256

Commit message: Layout.
Connections:
- net labels added: GPIO_G14, GPIO_H11, GPIO_J10
Changed lines of the file:
@@
 GPIO_D1
-Wire Wire Line
-	11150 2400 11750 2400
-Text Label 11750 2400 2    50   ~ 0
-GPIO_G4
 Wire Wire Line
 	11150 2500 11750 2500
@@
 Text Label 4200 8700 2    50   ~ 0
 GPIO_T15
+Text Label 2500 8200 0    50   ~ 0
+GPIO_P9
+Text Label 4200 8100 2    50   ~ 0
+GPIO_P8
+Text Label 2500 8100 0    50   ~ 0
+GPIO_T7
+Text Label 4200 8000 2    50   ~ 0
+GPIO_M8
+Text Label 2500 8000 0    50   ~ 0
+GPIO_N7
+Text Label 4200 7900 2    50   ~ 0
+GPIO_M7
+Text Label 2500 7900 0    50   ~ 0
+GPIO_N6
+Text Label 4200 7800 2    50   ~ 0
+GPIO_P6
+Text Label 2500 7800 0    50   ~ 0
+GPIO_N5
+Text Label 4200 7700 2    50   ~ 0
+GPIO_P5
+Text Label 2500 7700 0    50   ~ 0
+GPIO_P4
+Text Label 4200 7600 2    50   ~ 0
+GPIO_T6
+Text Label 2500 7600 0    50   ~ 0
+GPIO_R6
+Text Label 13000 7900 0    50   ~ 0
+GPIO_P7
+Text Label 13000 8300 0    50   ~ 0
+GPIO_T5
+Text Label 14700 8300 2    50   ~ 0
+GPIO_R5
+Text Label 13000 8200 0    50   ~ 0
+GPIO_R4
+Text Label 14700 8200 2    50   ~ 0
+GPIO_T3
+Text Label 13000 8100 0    50   ~ 0
+GPIO_R3
+Text Label 14700 8100 2    50   ~ 0
+GPIO_T2
+Text Label 13000 8000 0    50   ~ 0
+GPIO_R2
+Text Label 14700 8000 2    50   ~ 0
+GPIO_T1
+Text Label 9250 10000 0    50   ~ 0
+GPIO_E4
+Text Label 10950 10000 2    50   ~ 0
+GPIO_B2
+Text Label 10950 9900 2    50   ~ 0
+GPIO_B1
+Text Label 9250 9900 0    50   ~ 0
+GPIO_F5
+Text Label 10950 9800 2    50   ~ 0
+GPIO_C2
+Text Label 9250 9800 0    50   ~ 0
+GPIO_C1
+Text Label 10950 9700 2    50   ~ 0
+GPIO_D2
+Text Label 9250 9700 0    50   ~ 0
+GPIO_F4
+Text Label 10950 9600 2    50   ~ 0
+GPIO_D1
+Text Label 9250 9600 0    50   ~ 0
+GPIO_G5
+Text GLabel 14700 7700 2    50   BiDi ~ 0
+GPIO_G14
+Text GLabel 14700 7900 2    50   BiDi ~ 0
+GPIO_H11
+Text Label 13000 7800 0    50   ~ 0
+GPIO_K11
+Text GLabel 14700 7800 2    50   BiDi ~ 0
+GPIO_J10
+Text Label 10950 9500 2    50   ~ 0
+GPIO_E3
+Text Label 11750 2400 2    50   ~ 0
+GPIO_G4
+Wire Wire Line
+	11150 2400 11750 2400
+Text Label 9250 9500 0    50   ~ 0
+GPIO_G4
+Text Label 10950 9400 2    50   ~ 0
+GPIO_E2
+Text Label 9250 9400 0    50   ~ 0
+GPIO_H5
+Text Label 10950 9300 2    50   ~ 0
+GPIO_F3
+Text Label 9250 9300 0    50   ~ 0
+GPIO_G3
+Text Label 10950 9200 2    50   ~ 0
+GPIO_F2
+Text Label 9250 9200 0    50   ~ 0
+GPIO_H3
+Text Label 10950 9100 2    50   ~ 0
+GPIO_F1
+Text Label 9250 9100 0    50   ~ 0
+GPIO_H6
+Text Label 10950 9000 2    50   ~ 0
+GPIO_G2
+Text Label 9250 9000 0    50   ~ 0
+GPIO_H4
+Text Label 10950 8700 2    50   ~ 0
+GPIO_H2
+Text Label 9250 8700 0    50   ~ 0
+GPIO_J4
+Text Label 10950 8600 2    50   ~ 0
+GPIO_H1
+Text Label 9250 8600 0    50   ~ 0
+GPIO_J5
+Text Label 9250 8500 0    50   ~ 0
+GPIO_J2
+Text Label 10950 8500 2    50   ~ 0
+GPIO_J1
+Text Label 10950 8400 2    50   ~ 0
+GPIO_K3
+Text Label 9250 8400 0    50   ~ 0
+GPIO_K1
+Text Label 10950 8300 2    50   ~ 0
+GPIO_L1
+Text Label 9250 8300 0    50   ~ 0
+GPIO_L4
+Text Label 10950 8200 2    50   ~ 0
+GPIO_M1
+Text Label 9250 8200 0    50   ~ 0
+GPIO_K4
+Text Label 10950 8100 2    50   ~ 0
+GPIO_L3
+Text Label 9250 8100 0    50   ~ 0
+GPIO_L6
+Text Label 10950 8000 2    50   ~ 0
+GPIO_M2
+Text Label 9250 8000 0    50   ~ 0
+GPIO_K5
+Text Label 10950 7900 2    50   ~ 0
+GPIO_N2
+Text Label 9250 7900 0    50   ~ 0
+GPIO_L7
+Text Label 10950 7800 2    50   ~ 0
+GPIO_M3
+Text Label 9250 7800 0    50   ~ 0
+GPIO_M6
+Text Label 10950 7700 2    50   ~ 0
+GPIO_N3
+Text Label 9250 7700 0    50   ~ 0
+GPIO_L5
+Text Label 10950 7600 2    50   ~ 0
+GPIO_M4
+Text Label 9250 7600 0    50   ~ 0
+GPIO_P1
+Text Label 14700 7600 2    50   ~ 0
+GPIO_M5
+Text Label 13000 7600 0    50   ~ 0
+GPIO_P2
+Text Label 13000 7700 0    50   ~ 0
+GPIO_R1
+Text Label 9250 8900 0    50   ~ 0
+GPIO_N4
 $EndSCHEMATC

Commit message: Layout.
Connections:
- net GPIO_G14 is gone; now on net GPIO_P2: J3.10 (Pin_10)
- net GPIO_H11 is gone; now on net GPIO_P4: J3.14 (Pin_14)
- net GPIO_H12 is gone; now on net GPIO_M9: J4.46 (Pin_46)
- net GPIO_J11 is gone; now on net GPIO_K12: J4.55 (Pin_55)
- net GPIO_J12 is gone; now on net GPIO_K13: J4.56 (Pin_56)
- net GPIO_J13 is gone; now on net GPIO_L10: J4.44 (Pin_44)
- net DCDn: now also U4.P7 (IO2_22); no longer U4.N9 (IO2_23)
- net DSRn: now also U4.T7 (IO2_20); no longer U4.P10 (IO2_31)
- net DTRn: now also U4.P8 (IO2_17); no longer U4.N10 (IO2_32)
- net GPIO_J10: now also J4.41 (Pin_41); no longer J3.12 (Pin_12)
- net GPIO_J14: now also J4.42 (Pin_42); no longer J4.43 (Pin_43)
- net GPIO_K12: no longer J4.53 (Pin_53)
- net GPIO_K13: no longer J4.42 (Pin_42)
- net GPIO_K14: now also J4.37 (Pin_37); no longer J4.41 (Pin_41)
- net GPIO_L10: no longer J4.22 (Pin_22)
- net GPIO_L11: now also J4.51 (Pin_51); no longer J4.26 (Pin_26)
- net GPIO_L12: now also J4.53 (Pin_53); no longer J4.51 (Pin_51)
- net GPIO_L14: now also J4.35 (Pin_35); no longer J4.39 (Pin_39)
- net GPIO_L9: now also J4.43 (Pin_43); no longer J4.21 (Pin_21)
- net GPIO_M11: now also J4.49 (Pin_49); no longer J4.23 (Pin_23)
- net GPIO_M12: now also J4.52 (Pin_52); no longer J4.24 (Pin_24)
- net GPIO_M13: now also J4.27 (Pin_27); no longer J4.37 (Pin_37)
- net GPIO_M14: now also J4.30 (Pin_30); no longer J4.40 (Pin_40)
- net GPIO_M15: now also J4.33 (Pin_33); no longer J4.52 (Pin_52)
- net GPIO_M5: now also J4.8 (Pin_8); no longer J3.8 (Pin_8)
- net GPIO_M7: now also J4.10 (Pin_10); no longer J4.14 (Pin_14)
- net GPIO_M8: now also J4.12 (Pin_12); no longer J4.16 (Pin_16)
- net GPIO_M9: no longer J4.20 (Pin_20)
- net GPIO_N12: now also J4.50 (Pin_50); no longer J4.38 (Pin_38)
- net GPIO_N16: now also J4.29 (Pin_29); no longer J4.49 (Pin_49)
- net GPIO_N4: now also J4.7 (Pin_7); no longer J5.33 (Pin_33)
- net GPIO_N5: now also J3.16 (Pin_16); no longer J4.11 (Pin_11)
- net GPIO_N6: now also J4.9 (Pin_9); no longer J4.13 (Pin_13)
- net GPIO_N7: now also J4.11 (Pin_11); no longer J4.15 (Pin_15)
- net GPIO_P13: now also J4.18 (Pin_18); no longer J4.36 (Pin_36)
- net GPIO_P14: now also J4.24 (Pin_24); no longer J4.35 (Pin_35)
- net GPIO_P15: now also J4.26 (Pin_26); no longer J4.47 (Pin_47)
- net GPIO_P16: now also J4.28 (Pin_28); no longer J4.50 (Pin_50)
- net GPIO_P2: no longer J3.7 (Pin_7)
- net GPIO_P4: no longer J4.9 (Pin_9)
- net GPIO_P5: now also J3.18 (Pin_18); no longer J4.10 (Pin_10)
- net GPIO_P6: now also J3.19 (Pin_19); no longer J4.12 (Pin_12)
- net GPIO_R1: now also J3.8 (Pin_8); no longer J3.9 (Pin_9)
- net GPIO_R14: now also J4.20 (Pin_20); no longer J4.33 (Pin_33)
- net GPIO_R15: now also J4.22 (Pin_22); no longer J4.45 (Pin_45)
- net GPIO_R16: now also J4.25 (Pin_25); no longer J4.48 (Pin_48)
- net GPIO_R2: now also J3.9 (Pin_9); no longer J3.15 (Pin_15)
- net GPIO_R3: now also J3.11 (Pin_11); no longer J3.17 (Pin_17)
- net GPIO_R4: now also J3.15 (Pin_15); no longer J3.19 (Pin_19)
- net GPIO_R5: now also J3.17 (Pin_17); no longer J3.22 (Pin_22)
- net GPIO_R6: now also J3.22 (Pin_22); no longer J4.7 (Pin_7)
- net GPIO_T1: now also J3.7 (Pin_7); no longer J3.16 (Pin_16)
- net GPIO_T11: now also J4.13 (Pin_13); no longer J4.25 (Pin_25)
- net GPIO_T13: now also J4.17 (Pin_17); no longer J4.28 (Pin_28)
- net GPIO_T14: now also J4.19 (Pin_19); no longer J4.27 (Pin_27)
- net GPIO_T15: now also J4.21 (Pin_21); no longer J4.30 (Pin_30)
- net GPIO_T16: now also J4.23 (Pin_23); no longer J4.29 (Pin_29)
- net GPIO_T2: now also J3.12 (Pin_12); no longer J3.18 (Pin_18)
- net GPIO_T3: now also J3.13 (Pin_13); no longer J3.20 (Pin_20)
- net GPIO_T5: now also J3.20 (Pin_20); no longer J3.21 (Pin_21)
- net GPIO_T6: now also J3.21 (Pin_21); no longer J4.8 (Pin_8)
- net ICE_CLK_12MHZ: now also U4.R9 (GBIN5/IO2_26); no longer U4.J3 (GBIN6/IO3_13A)
- net RS232_RX_TTL: now also U4.N9 (IO2_23); no longer U4.T10 (IO2_33)
- net RS232_TX_TTL: now also U4.P9 (IO2_28); no longer U4.R10 (IO2_29)
- net GPIO_K9: now reaches U4.K9 (GBIN4/IO2_27)
- net GPIO_K9: now also J5.33 (Pin_33)
- net ICE_CLK_26.601712MHz: now reaches U4.G1 (GBIN7/IO3_12B)
- net GPIO_K11 renamed ICE_M2
- net ICE_M2: no longer J3.11 (Pin_11)
- removed net GPIO_P7: J3.13 (Pin_13), U4.P7 (IO2_22)
- removed net GPIO_P8: J4.18 (Pin_18), U4.P8 (IO2_17)
- removed net GPIO_P9: J4.19 (Pin_19), U4.P9 (IO2_28)
- removed net GPIO_T7: J4.17 (Pin_17), U4.T7 (IO2_20)
- new net GPIO_J15: J4.48 (Pin_48)
- new net GPIO_J16: J4.47 (Pin_47)
- new net GPIO_K15: J4.40 (Pin_40)
- new net GPIO_K16: J4.39 (Pin_39)
- new net GPIO_L16: J4.38 (Pin_38)
- new net GPIO_M16: J4.36 (Pin_36)
- new net GPIO_N10: J4.45 (Pin_45), U4.N10 (IO2_32)
- new net GPIO_P10: J4.14 (Pin_14), U4.P10 (IO2_31)
- new net GPIO_R10: J4.15 (Pin_15), U4.R10 (IO2_29)
- new net GPIO_T10: J4.16 (Pin_16), U4.T10 (IO2_33)
- no-connect marks 3 -> 1

Commit message: Layout. Cleaned up nes connector footprints. Adjusted LED (D1) series resistor. Adjusted the voltage divider to BCBUS7 on FT2232H. Set pull up resistor to CDONE to 10k.
Parts:
- R36: value R_TBD -> R10K; symbol icenes-library:R_TBD -> icenes-library:R10K; Manufacturer (none) -> Yageo; Part number (none) -> RC0603FR-0710KL; Resistance (none) -> 10k
Other:
- note added: "Rough estimation for max resistance \nis about 13k.\nTry with 10k to begin with.\nIf 10k does no work move down to \n6.04k, 4.7k, 2.2k. 1.54k. 698, 200."
Changed lines of the file:
@@
 Text Label 5000 1600 2    50   ~ 0
 GPIO_P4
-Wire Wire Line
-	3100 4200 2500 4200
-Text Label 2500 4200 0    50   ~ 0
+Text Label 2700 4200 0    50   ~ 0
 GPIO_P13
-Wire Wire Line
-	3100 4100 2500 4100
 $Comp
 L icenes-library:Conn_02x31_Odd_Even J4
@@
 	10600 8800 11100 8800
 $Comp
-L icenes-library:R_TBD R36
+L icenes-library:R10K R36
 U 1 1 5DA26BEC
 P 1300 4200
 F 0 "R36" V 1300 4270 50  0000 L CNN
-F 1 "R_TBD" H 1300 4100 50  0001 C CNN
+F 1 "R10K" H 1300 4100 50  0001 C CNN
 F 2 "Resistor_SMD:R_0603_1608Metric_Pad1.05x0.95mm_HandSolder" V 1300 4200 50  0001 C CNN
-F 3 "" V 1300 4200 50  0001 C CNN
+F 3 "https://www.mouser.se/datasheet/2/447/PYu-RC_Group_51_RoHS_L_10-1527934.pdf" V 1300 4200 50  0001 C CNN
+F 4 "10k" V 1375 4350 50  0000 C CNN "Resistance"
+F 5 "Yageo" V 1300 4200 50  0001 C CNN "Manufacturer"
+F 6 "RC0603FR-0710KL" V 1300 4200 50  0001 C CNN "Part number"
 	1    1300 4200
 	0    1    1    0
@@
 Wire Wire Line
 	2250 9600 3100 9600
-Text GLabel 2500 4100 0    50   Output ~ 0
+Text GLabel 2675 4100 0    50   Output ~ 0
 ICE_M2
+Text Notes 525  4300 0    25   ~ 0
+Rough estimation for max resistance \nis about 13k.\nTry with 10k to begin with.\nIf 10k does no work move down to \n6.04k, 4.7k, 2.2k. 1.54k. 698, 200.
+Wire Wire Line
+	3100 4200 2700 4200
+Wire Wire Line
+	2675 4100 3100 4100
 $EndSCHEMATC
