File: hw/icenes-nes-connector.sch (KiCad schematic (older format))
At the start: 22 parts, among them J6 NES-Connector-72pin, U10 74ALVC164245, U11 74ALVC164245, U12 74ALVC164245, U13 74ALVC164245

Commit message: Rough board layout.
Parts:
- J6: footprint icenes-library:DIP-72-NES-CONNECTOR -> icenes-library:DIP-72-NES-CONNECTOR-2
Changed lines of the file:
@@
 F 0 "J6" H 12975 2065 50  0000 C CNN
 F 1 "NES-Connector-72pin" H 12975 1974 50  0000 C CNN
-F 2 "icenes-library:DIP-72-NES-CONNECTOR" H 12950 1950 50  0001 C CNN
+F 2 "icenes-library:DIP-72-NES-CONNECTOR-2" H 12950 1950 50  0001 C CNN
 F 3 "" H 12950 1950 50  0001 C CNN
 	1    12950 1950

Commit message: Layout.
Connections:
- net ICE_PPU_A10: now also U10.35 (2A2); no longer U10.33 (2A3)
- net ICE_PPU_A11: now also U10.33 (2A3); no longer U10.32 (2A4)
- net ICE_PPU_A12: now also U10.36 (2A1); no longer U10.30 (2A5)
- net ICE_PPU_A13: now also U10.37 (1A8); no longer U10.29 (2A6)
- net ICE_PPU_A7: now also U10.29 (2A6); no longer U10.37 (1A8)
- net ICE_PPU_A8: now also U10.30 (2A5); no longer U10.36 (2A1)
- net ICE_PPU_A9: now also U10.32 (2A4); no longer U10.35 (2A2)
- net NES_PPU_A10: now also U10.14 (2B2); no longer U10.16 (2B3)
- net NES_PPU_A11: now also U10.16 (2B3); no longer U10.17 (2B4)
- net NES_PPU_A12: now also U10.13 (2B1); no longer U10.19 (2B5)
- net NES_PPU_A13: now also U10.12 (1B8); no longer U10.20 (2B6)
- net NES_PPU_A7: now also U10.20 (2B6); no longer U10.12 (1B8)
- net NES_PPU_A8: now also U10.19 (2B5); no longer U10.13 (2B1)
- net NES_PPU_A9: now also U10.17 (2B4); no longer U10.14 (2B2)
Changed lines of the file:
@@
 	1850 3000 1750 3000
-Wire Wire Line
-	1850 3100 1750 3100
-Wire Wire Line
-	1850 3200 1750 3200
-Wire Wire Line
-	1850 3300 1750 3300
-Wire Wire Line
-	1850 3400 1750 3400
-Wire Wire Line
-	1850 3500 1750 3500
-Wire Wire Line
-	1850 3600 1750 3600
-Wire Wire Line
-	1850 3700 1750 3700
 Wire Wire Line
 	12100 5650 12000 5650
@@
 Text GLabel 1700 4100 0    50   Input ~ 0
 ~PPU_ADDR_OE
-Text GLabel 1750 3700 0    50   Input ~ 0
-ICE_PPU_A13
-Text GLabel 1750 3600 0    50   Input ~ 0
-ICE_PPU_A12
-Text GLabel 1750 3500 0    50   Input ~ 0
-ICE_PPU_A11
-Text GLabel 1750 3400 0    50   Input ~ 0
-ICE_PPU_A10
-Text GLabel 1750 3300 0    50   Input ~ 0
-ICE_PPU_A9
-Text GLabel 1750 3200 0    50   Input ~ 0
-ICE_PPU_A8
-Text GLabel 1750 3100 0    50   Input ~ 0
-ICE_PPU_A7
 Text GLabel 1750 3000 0    50   Input ~ 0
 ICE_PPU_A6
@@
 	3050 3100 3650 3100
 Wire Wire Line
-	3050 3200 3650 3200
-Wire Wire Line
-	3050 3300 3650 3300
-Wire Wire Line
-	3050 3400 3650 3400
-Wire Wire Line
-	3050 3500 3650 3500
-Wire Wire Line
-	3050 3600 3650 3600
-Wire Wire Line
-	3050 3700 3650 3700
-Wire Wire Line
 	3050 3800 3650 3800
 Wire Wire Line
@@
 Wire Wire Line
 	13850 2950 14500 2950
-Wire Wire Line
-	13850 3050 14500 3050
-Wire Wire Line
-	13850 3150 14500 3150
 Wire Wire Line
 	13850 3250 14500 3250
@@
 NES_PPU_A6
 Text Label 3650 3100 2    50   ~ 0
-NES_PPU_A7
-Text Label 3650 3200 2    50   ~ 0
-NES_PPU_A8
-Text Label 3650 3300 2    50   ~ 0
-NES_PPU_A9
-Text Label 3650 3400 2    50   ~ 0
-NES_PPU_A10
-Text Label 3650 3500 2    50   ~ 0
-NES_PPU_A11
-Text Label 3650 3600 2    50   ~ 0
-NES_PPU_A12
-Text Label 3650 3700 2    50   ~ 0
 NES_PPU_A13
 Text Label 3650 3800 2    50   ~ 0
@@
 Text Label 14500 2950 2    50   ~ 0
 NES_PPU_A12
-Text Label 14500 3050 2    50   ~ 0
-NES_PPU_A10
-Text Label 14500 3150 2    50   ~ 0
-NES_PPU_A11
 Text Label 14500 3250 2    50   ~ 0
 NES_PPU_A9
@@
 Wire Wire Line
 	7150 4300 7150 4400
+Text GLabel 1750 3100 0    50   Input ~ 0
+ICE_PPU_A13
+Wire Wire Line
+	1850 3100 1750 3100
+Text Label 3650 3500 2    50   ~ 0
+NES_PPU_A9
+Wire Wire Line
+	3050 3500 3650 3500
+Text Label 3650 3300 2    50   ~ 0
+NES_PPU_A10
+Wire Wire Line
+	3050 3300 3650 3300
+Text Label 3650 3400 2    50   ~ 0
+NES_PPU_A11
+Wire Wire Line
+	3050 3400 3650 3400
+Text Label 3650 3600 2    50   ~ 0
+NES_PPU_A8
+Wire Wire Line
+	3050 3600 3650 3600
+Text Label 3650 3700 2    50   ~ 0
+NES_PPU_A7
+Wire Wire Line
+	3050 3700 3650 3700
+Text Label 3650 3200 2    50   ~ 0
+NES_PPU_A12
+Wire Wire Line
+	3050 3200 3650 3200
+Wire Wire Line
+	1850 3300 1750 3300
+Text GLabel 1750 3300 0    50   Input ~ 0
+ICE_PPU_A10
+Wire Wire Line
+	1850 3500 1750 3500
+Text GLabel 1750 3500 0    50   Input ~ 0
+ICE_PPU_A9
+Wire Wire Line
+	1850 3400 1750 3400
+Text GLabel 1750 3400 0    50   Input ~ 0
+ICE_PPU_A11
+Wire Wire Line
+	1850 3600 1750 3600
+Text GLabel 1750 3600 0    50   Input ~ 0
+ICE_PPU_A8
+Wire Wire Line
+	1850 3700 1750 3700
+Text GLabel 1750 3700 0    50   Input ~ 0
+ICE_PPU_A7
+Wire Wire Line
+	1850 3200 1750 3200
+Text GLabel 1750 3200 0    50   Input ~ 0
+ICE_PPU_A12
+Text Label 14500 3150 2    50   ~ 0
+NES_PPU_A11
+Wire Wire Line
+	13850 3150 14500 3150
+Text Label 14500 3050 2    50   ~ 0
+NES_PPU_A10
+Wire Wire Line
+	13850 3050 14500 3050
 $EndSCHEMATC

Commit message: Layout.  - Changed footprint of the nes connector from 2.54mm pitch and 5.08mm row pitch to 2.5mm pitch and 0.5mm row pitch.
Parts:
- J6: footprint icenes-library:DIP-72-NES-CONNECTOR-2 -> icenes-library:DIP-72-NES-CONNECTOR-3
Changed lines of the file:
@@
 F 0 "J6" H 12975 2065 50  0000 C CNN
 F 1 "NES-Connector-72pin" H 12975 1974 50  0000 C CNN
-F 2 "icenes-library:DIP-72-NES-CONNECTOR-2" H 12950 1950 50  0001 C CNN
+F 2 "icenes-library:DIP-72-NES-CONNECTOR-3" H 12950 1950 50  0001 C CNN
 F 3 "" H 12950 1950 50  0001 C CNN
 	1    12950 1950

Commit message: Layout. Cleaned up nes connector footprints. Adjusted LED (D1) series resistor. Adjusted the voltage divider to BCBUS7 on FT2232H. Set pull up resistor to CDONE to 10k.
Parts:
- J6: footprint icenes-library:DIP-72-NES-CONNECTOR-3 -> icenes-library:DIP-72-NES-CONNECTOR
Changed lines of the file:
@@
 F 0 "J6" H 12975 2065 50  0000 C CNN
 F 1 "NES-Connector-72pin" H 12975 1974 50  0000 C CNN
-F 2 "icenes-library:DIP-72-NES-CONNECTOR-3" H 12950 1950 50  0001 C CNN
+F 2 "icenes-library:DIP-72-NES-CONNECTOR" H 12950 1950 50  0001 C CNN
 F 3 "" H 12950 1950 50  0001 C CNN
 	1    12950 1950
